File: hardware/project/ETH1CDMM2/Connector.kicad_sch (KiCad schematic)
At the start: 7 parts, among them J1001 C64AC, K1201 HE3621A0510, K1202 HE3621A0510, K1203 HE3621A0510, K1204 HE3621A0510, K1205 HE3621A0510, K1206 HE3621A0510

Commit message: Hardware development
Parts:
- K1201, K1202, K1203, K1204, K1205, K1206: footprint (none) -> ETH1CDMM2:HE360_x-5050462-8
Connections:
- net +24VF renamed +24V
- net DGNDF renamed GNDPWR
Changed lines of the file:
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@@
     (effects (font (size 1.27 1.27)) (justify right))
   )
-  (hierarchical_label "OUT_REL[0..5]" (shape input) (at 265.43 58.42 0) (fields_autoplaced)
+  (hierarchical_label "OUT_REL[0..5]" (shape bidirectional) (at 265.43 58.42 0) (fields_autoplaced)
     (effects (font (size 1.27 1.27)) (justify left))
   )
@@
       (effects (font (size 1.27 1.27)))
     )
-    (property "Footprint" "" (at 93.98 20.32 0)
+    (property "Footprint" "ETH1CDMM2:HE360_x-5050462-8" (at 93.98 20.32 0)
       (effects (font (size 1.27 1.27)) hide)
     )
@@
       (effects (font (size 1.27 1.27)) (justify left))
     )
-    (property "Footprint" "" (at 177.8 41.91 0)
+    (property "Footprint" "ETH1CDMM2:HE360_x-5050462-8" (at 177.8 41.91 0)
       (effects (font (size 1.27 1.27)) hide)
     )
@@
       (effects (font (size 1.27 1.27)))
     )
-    (property "Footprint" "" (at 93.98 55.88 0)
+    (property "Footprint" "ETH1CDMM2:HE360_x-5050462-8" (at 93.98 55.88 0)
       (effects (font (size 1.27 1.27)) hide)
     )
@@
       (effects (font (size 1.27 1.27)) (justify left))
     )
-    (property "Footprint" "" (at 234.95 41.91 0)
+    (property "Footprint" "ETH1CDMM2:HE360_x-5050462-8" (at 234.95 41.91 0)
       (effects (font (size 1.27 1.27)) hide)
     )
@@
       (effects (font (size 1.27 1.27)))
     )
-    (property "Footprint" "" (at 93.98 29.21 0)
+    (property "Footprint" "ETH1CDMM2:HE360_x-5050462-8" (at 93.98 29.21 0)
       (effects (font (size 1.27 1.27)) hide)
     )
@@
       (effects (font (size 1.27 1.27)) (justify left))
     )
-    (property "Footprint" "" (at 196.85 41.91 0)
+    (property "Footprint" "ETH1CDMM2:HE360_x-5050462-8" (at 196.85 41.91 0)
       (effects (font (size 1.27 1.27)) hide)
     )
@@
       (effects (font (size 1.27 1.27)))
     )
-    (property "Footprint" "" (at 93.98 64.77 0)
+    (property "Footprint" "ETH1CDMM2:HE360_x-5050462-8" (at 93.98 64.77 0)
       (effects (font (size 1.27 1.27)) hide)
     )
@@
       (effects (font (size 1.27 1.27)) (justify left))
     )
-    (property "Footprint" "" (at 252.73 41.91 0)
+    (property "Footprint" "ETH1CDMM2:HE360_x-5050462-8" (at 252.73 41.91 0)
       (effects (font (size 1.27 1.27)) hide)
     )
@@
       (effects (font (size 1.27 1.27)))
     )
-    (property "Footprint" "" (at 93.98 38.1 0)
+    (property "Footprint" "ETH1CDMM2:HE360_x-5050462-8" (at 93.98 38.1 0)
       (effects (font (size 1.27 1.27)) hide)
     )
@@
       (effects (font (size 1.27 1.27)) (justify left))
     )
-    (property "Footprint" "" (at 215.9 41.91 0)
+    (property "Footprint" "ETH1CDMM2:HE360_x-5050462-8" (at 215.9 41.91 0)
       (effects (font (size 1.27 1.27)) hide)
     )
@@
       (effects (font (size 1.27 1.27)))
     )
-    (property "Footprint" "" (at 93.98 46.99 0)
+    (property "Footprint" "ETH1CDMM2:HE360_x-5050462-8" (at 93.98 46.99 0)
       (effects (font (size 1.27 1.27)) hide)
     )
@@
       (effects (font (size 1.27 1.27)) (justify left))
     )
-    (property "Footprint" "" (at 158.75 41.91 0)
+    (property "Footprint" "ETH1CDMM2:HE360_x-5050462-8" (at 158.75 41.91 0)
       (effects (font (size 1.27 1.27)) hide)
     )
@@
         (path "/be7d1fbf-8f6a-4ef0-a932-f9076baf5f6b/00000000-0000-0000-0000-000060bf6da7"
           (reference "K1204") (unit 2)
-        )
-      )
-    )
-  )
-  (symbol (lib_id "ETH1CDMM2:+24VF") (at 121.92 180.34 90) (unit 1)
-    (in_bom yes) (on_board yes) (dnp no)
-    (property "Reference" "#PWR01204" (at 125.73 180.34 0)
-      (effects (font (size 1.27 1.27)) hide)
-    )
-    (property "Value" "+24VF" (at 118.6942 179.959 90)
-      (effects (font (size 1.27 1.27)) (justify left))
-    )
-    (property "Footprint" "" (at 121.92 180.34 0)
-      (effects (font (size 1.27 1.27)) hide)
-    )
-    (property "Datasheet" "" (at 121.92 180.34 0)
-      (effects (font (size 1.27 1.27)) hide)
-    )
-    (pin "1")
-    (instances
-      (project "ETH1CDMM2"
-        (path "/be7d1fbf-8f6a-4ef0-a932-f9076baf5f6b/00000000-0000-0000-0000-000060bf6da7"
-          (reference "#PWR01204") (unit 1)
-        )
-      )
-    )
-  )
-  (symbol (lib_id "ETH1CDMM2:DGNDF") (at 121.92 160.02 270) (unit 1)
-    (in_bom yes) (on_board yes) (dnp no)
-    (property "Reference" "#PWR01203" (at 115.57 160.02 0)
-      (effects (font (size 1.27 1.27)) hide)
-    )
-    (property "Value" "DGNDF" (at 118.6942 160.147 90)
-      (effects (font (size 1.27 1.27)) (justify right))
-    )
-    (property "Footprint" "" (at 121.92 160.02 0)
-      (effects (font (size 1.27 1.27)) hide)
-    )
-    (property "Datasheet" "" (at 121.92 160.02 0)
-      (effects (font (size 1.27 1.27)) hide)
-    )
-    (pin "1")
-    (instances
-      (project "ETH1CDMM2"
-        (path "/be7d1fbf-8f6a-4ef0-a932-f9076baf5f6b/00000000-0000-0000-0000-000060bf6da7"
-          (reference "#PWR01203") (unit 1)
         )
       )
@@
         )
       )
+    )
+  )
+  (symbol (lib_id "power:GNDPWR") (at 121.92 160.02 270) (unit 1)
+    (in_bom yes) (on_board yes) (dnp no)
+    (property "Reference" "#PWR01004" (at 116.84 160.02 0)
+      (effects (font (size 1.27 1.27)) hide)
+    )
+    (property "Value" "GNDPWR" (at 115.57 160.02 90)
+      (effects (font (size 1.27 1.27)))
+    )
+    (property "Footprint" "" (at 120.65 160.02 0)
+      (effects (font (size 1.27 1.27)) hide)
+    )
+    (property "Datasheet" "" (at 120.65 160.02 0)
+      (effects (font (size 1.27 1.27)) hide)
+    )
+    (pin "1")
+    (instances
+      (project "ETH1CDMM2"
+        (path "/be7d1fbf-8f6a-4ef0-a932-f9076baf5f6b/00000000-0000-0000-0000-0000602ff78d"
+          (reference "#PWR01004") (unit 1)
+        )
+        (path "/be7d1fbf-8f6a-4ef0-a932-f9076baf5f6b/00000000-0000-0000-0000-000060bf6da7"
+          (reference "#PWR01203") (unit 1)
+        )
+      )
+    )
+  )
+  (symbol (lib_id "power:+24V") (at 121.92 180.34 90) (unit 1)
+    (in_bom yes) (on_board yes) (dnp no)
+    (property "Reference" "#PWR01204" (at 125.73 180.34 0)
+      (effects (font (size 1.27 1.27)) hide)
+    )
+    (property "Value" "+24V" (at 118.11 180.34 90)
+      (effects (font (size 1.27 1.27)) (justify left))
+    )
+    (property "Footprint" "" (at 121.92 180.34 0)
+      (effects (font (size 1.27 1.27)) hide)
+    )
+    (property "Datasheet" "" (at 121.92 180.34 0)
+      (effects (font (size 1.27 1.27)) hide)
+    )
+    (pin "1")
+    (instances
+      (project "ETH1CDMM2"
+        (path "/be7d1fbf-8f6a-4ef0-a932-f9076baf5f6b/00000000-0000-0000-0000-000060bf6da7"
+          (reference "#PWR01204") (unit 1)
+        )
+      )
