File: hardware/project/ETH1CDMM2/FPGA.kicad_sch (KiCad schematic)
At the start: 64 parts, among them J401 Conn_01x04_Male, J402 Conn_02x05, Q401 BC857, U401 SN74LVC1T45DBV, U402 SN74LVC1T45DBV, U403 ICE40HX4K-TQ144, U404 SN74LVC1T45DBV, U405 SN74LVC1T45DBV, U406 SN74LVC1T45DBV, U407 SN74LVC1T45DBV, U408 ASDMB-100.000MHZ, U409 MT25QL128ABA1ESE

Commit message: Hardware development
Parts:
- C401, C402, C403, C404, C405, C406, C407, C408, C409, C410, C411, C412, C413, C414, C415, C416, C417, C418, C419, C420, C421, C422, C423, C424, C425, C426, C428, C430: footprint Capacitor_SMD:C_0603_1608Metric_Pad1.05x0.95mm_HandSolder -> Capacitor_SMD:C_0603_1608Metric_Pad1.08x0.95mm_HandSolder
- C427, C429: footprint Capacitor_SMD:C_0805_2012Metric_Pad1.15x1.40mm_HandSolder -> Capacitor_SMD:C_0805_2012Metric_Pad1.18x1.45mm_HandSolder
- R401, R402, R403, R404, R405, R406, R407, R408, R409, R410, R411, R412, R413, R414, R415, R416, R417, R418, R419: footprint Resistor_SMD:R_0603_1608Metric_Pad1.05x0.95mm_HandSolder -> Resistor_SMD:R_0603_1608Metric_Pad0.98x0.95mm_HandSolder
Connections:
- net FPGA_AD_RFS_OPT: no longer names the net of U403.8 (IOL_4B)
- no-connect marks 78 -> 79
