File: hardware/project/ETH1CDMM2/MCU.kicad_sch (KiCad schematic)
At the start: 42 parts, among them J601 Conn_02x01, J602 20021111-00010T4LF, U601 HDC1080, U602 STM32H743ZI, U603 24LC08B-E/MS, Y601 NX3225GD-8MHZ-STD-CRA-3

Commit message: Hardware development
Parts:
- C601, C602, C603, C604, C605, C606, C607, C609, C611, C612, C613, C614, C615, C616, C617, C618, C619, C620, C621, C622: footprint Capacitor_SMD:C_0603_1608Metric_Pad1.05x0.95mm_HandSolder -> Capacitor_SMD:C_0603_1608Metric_Pad1.08x0.95mm_HandSolder
- C608, C610: footprint Capacitor_SMD:C_0805_2012Metric_Pad1.15x1.40mm_HandSolder -> Capacitor_SMD:C_0805_2012Metric_Pad1.18x1.45mm_HandSolder
Connections:
- net SPI4_SCK: now reaches U602.1 (PE2,TRACECLK,SPI4_SCK,SAI1_MCLK_A,QUADSPI_BK1_IO2,ETH_MII_TXD3,FMC_A23,EVENTOUT)
- net SPI4_NSS: now reaches U602.3 (PE4,TRACED1,SPI4_NSS,SAI1_FS_A,DFSDM1_DATIN3,FMC_A20,DCMI_D4,LCD_B0,EVENTOUT)
- net SPI4_MOSI: now reaches U602.5 (PE6,TRACED3,TIM1_BKIN2,TIM9_CH2,SPI4_MOSI,SAI1_SD_A,SAI2_MCLK_B,FMC_A22,DCMI_D7,LCD_G1,EVENTOUT)
- no-connect marks 44 -> 41
