File: hardware/project/ETH1CDMM2/ADC.kicad_sch (KiCad schematic)
At the start: 79 parts, among them Q201 BC847, Q203 BC847, U203 DG419xY

Commit message: Hardware development
Parts:
- removed C201: 10p, Capacitor_SMD:C_0603_1608Metric_Pad1.05x0.95mm_HandSolder, symbol Device:C
- removed D201: 1N4148W, Diode_SMD:D_SOD-123, symbol Diode:1N4148W
- removed K? (x2): 9012, ETH1CDMM2:9012, symbol ETH1CDMM2:9012
- removed Q201: BC847, Package_TO_SOT_SMD:SOT-23, symbol Transistor_BJT:BC847
- removed R201: 10k, Resistor_SMD:R_0603_1608Metric_Pad1.05x0.95mm_HandSolder, symbol Device:R
- C202, C203, C204, C205, C206, C207, C208, C209, C210, C211, C212, C213, C215, C216, C217, C218, C219, C220, C221, C223, C224: footprint Capacitor_SMD:C_0603_1608Metric_Pad1.05x0.95mm_HandSolder -> Capacitor_SMD:C_0603_1608Metric_Pad1.08x0.95mm_HandSolder
- C222: footprint Capacitor_SMD:C_0603_1608Metric_Pad1.05x0.95mm_HandSolder -> Capacitor_SMD:C_0603_1608Metric_Pad1.08x0.95mm_HandSolder; now not fitted
- R203, R205, R207, R208, R209, R211, R212, R217, R218, R219, R220, R223: footprint Resistor_SMD:R_0603_1608Metric_Pad1.05x0.95mm_HandSolder -> Resistor_SMD:R_0603_1608Metric_Pad0.98x0.95mm_HandSolder
- U203: value DG419xY -> DG419DY+
- U? (x5): value DG211B -> DG211DY+
- U? (x3): value OPA2192 -> OPA2192ID
- U?: value OPA140 -> OPA140AID
- U? (x2): value OPA177 -> OPA177GS
- U?: value OPA192 -> OPA192ID
- U?: value LM311 -> LM311DR
Other:
- moved on the sheet: C202, C203, C204, C205, C206, C207, C208, C209, C210, C212, C213, C216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

Commit message: Hardware design
Parts:
- D201: renamed from D202; footprint Diode_SMD:D_SOD-523 -> Diode_SMD:D_SOD-123
- Q?: value MMBTA55 -> MMBTA55-TP
- R203: renamed from R202; footprint Resistor_SMD:R_0603_1608Metric_Pad1.05x0.95mm_HandSolder -> Resistor_SMD:R_0603_1608Metric_Pad0.98x0.95mm_HandSolder
- R204: footprint Resistor_SMD:R_0603_1608Metric_Pad1.05x0.95mm_HandSolder -> Resistor_SMD:R_0603_1608Metric_Pad0.98x0.95mm_HandSolder
- R205: renamed from R206; footprint Resistor_SMD:R_0603_1608Metric_Pad1.05x0.95mm_HandSolder -> Resistor_SMD:R_0603_1608Metric_Pad0.98x0.95mm_HandSolder
- R209: renamed from R210; footprint Resistor_SMD:R_0603_1608Metric_Pad1.05x0.95mm_HandSolder -> Resistor_SMD:R_0603_1608Metric_Pad0.98x0.95mm_HandSolder
- R212: renamed from R213; footprint Resistor_SMD:R_1206_3216Metric_Pad1.42x1.75mm_HandSolder -> Resistor_SMD:R_1206_3216Metric_Pad1.30x1.75mm_HandSolder
- R213: renamed from R214; footprint Resistor_SMD:R_0603_1608Metric_Pad1.05x0.95mm_HandSolder -> Resistor_SMD:R_0603_1608Metric_Pad0.98x0.95mm_HandSolder
- R214: renamed from R215; footprint Resistor_SMD:R_0603_1608Metric_Pad1.05x0.95mm_HandSolder -> Resistor_SMD:R_0603_1608Metric_Pad0.98x0.95mm_HandSolder
- R215: renamed from R216; footprint Resistor_SMD:R_0603_1608Metric_Pad1.05x0.95mm_HandSolder -> Resistor_SMD:R_0603_1608Metric_Pad0.98x0.95mm_HandSolder
- R220: renamed from R221; footprint Resistor_SMD:R_0603_1608Metric_Pad1.05x0.95mm_HandSolder -> Resistor_SMD:R_0603_1608Metric_Pad0.98x0.95mm_HandSolder
- R221: renamed from R222; footprint Resistor_SMD:R_0603_1608Metric_Pad1.05x0.95mm_HandSolder -> Resistor_SMD:R_0603_1608Metric_Pad0.98x0.95mm_HandSolder
- R223: renamed from R224; footprint Resistor_SMD:R_0603_1608Metric_Pad1.05x0.95mm_HandSolder -> Resistor_SMD:R_0603_1608Metric_Pad0.98x0.95mm_HandSolder
- R224: renamed from R225; footprint Resistor_SMD:R_0603_1608Metric_Pad1.05x0.95mm_HandSolder -> Resistor_SMD:R_0603_1608Metric_Pad0.98x0.95mm_HandSolder
- R225: renamed from R226; footprint Resistor_SMD:R_0603_1608Metric_Pad1.05x0.95mm_HandSolder -> Resistor_SMD:R_0603_1608Metric_Pad0.98x0.95mm_HandSolder
- renumbered C202 to C201, C203 to C202, C204 to C203, C205 to C204, C206 to C205, C207 to C206, C208 to C207, C209 to C208, C210 to C209, C212 to C210, C213 to C212, C214 to C213, C215 to C214, C216 to C215, C217 to C216, C218 to C217, C219 to C218, C220 to C219, C221 to C220, C223 to C221, C224 to C223, D203 to D202, D204 to D203, D205 to D204, Q203 to Q201, R203 to R201, R205 to R202, R207 to R206, R208 to R207, R209 to R208, R211 to R210, R212 to R211, R217 to R216, R218 to R217, R219 to R218, R220 to R219, R223 to R222
