File: hardware/project/ETH1CDMM2/FrontEnd.kicad_sch (KiCad schematic)
At the start: 24 parts, among them Q601 BC847, Q602 BC857, U601 DG211B, U602 DG211B, U608 LTC1052, U609 AD711, U610 AD711, U611 TL431DBZ, U612 TL431DBZ, U613 LT5400-9k-1k

Commit message: Hardware development
Parts:
- removed C625: 4n7, Capacitor_SMD:C_0603_1608Metric_Pad1.05x0.95mm_HandSolder, symbol Device:C
- removed U613: LT5400-9k-1k, Package_SO:MSOP-8-1EP_3x3mm_P0.65mm_EP1.73x1.85mm_ThermalVias, symbol ADC_TEST:LT5400-9k-1k
- added C1401, C1402, C1403, C1404, C1405, C1406, C1407, C1408, C1409, C1410: 100n, Capacitor_SMD:C_0603_1608Metric_Pad1.08x0.95mm_HandSolder, symbol Device:C
- added R1402: RG2012N-184-W-T1, symbol Device:R
- added U1403: DG211DY+, Package_SO:SOIC-16_3.9x9.9mm_P1.27mm, symbol ETH1CDMM2:DG211
- added U1404: LT5400-8, Package_SO:MSOP-8-1EP_3x3mm_P0.65mm_EP1.73x1.85mm_ThermalVias, symbol ETH1CDMM2:LT5400-9k-1k_Split
- C617, C620, C624: footprint Capacitor_SMD:C_0603_1608Metric_Pad1.05x0.95mm_HandSolder -> Capacitor_SMD:C_0603_1608Metric_Pad1.08x0.95mm_HandSolder
- R624, R625, R626, R627, R628, R629: footprint Resistor_SMD:R_0805_2012Metric_Pad1.15x1.40mm_HandSolder -> Resistor_SMD:R_0805_2012Metric_Pad1.20x1.40mm_HandSolder
- U601, U602: value DG211B -> DG211DY+; symbol ADC_TEST:DG211 -> ETH1CDMM2:DG211
- U608: value LTC1052 -> LTC1052CN8#PBF; symbol ADC_TEST:LTC1052 -> ETH1CDMM2:LTC1052
- U609, U610: value AD711 -> AD711JRZ; symbol ADC_TEST:AD711 -> ETH1CDMM2:AD711
Connections:
- net FE_GND is gone; now on net +5VF: U602.8
- net +18VF: now also C1401.1, C1402.1, C1403.1, C1404.1, U1403.13 (V+)
- net +5VF: now also C1405.1, C1406.1, U1403.12 (VL)
- net -14VF: now also C1407.1, C1408.1, C1409.1, U1403.4 (V-)
- net -18VF: now also C1410.1
- net ADIN: now also U602.3, R1402.1; no longer U602.15
- net AGNDF: now also C1401.2, C1402.2, C1403.2, C1404.2, C1405.2, C1406.2, C1407.2, C1408.2, C1409.2, C1410.2, U1403.10, U1403.5 (GND), U1403.6, U1404.2 (R2.1), U1404.9 (R1.2); no longer U602.6
- net at R623.2, U608.2 (-), U609.2 (-): now also U602.10, U602.15, U602.2; no longer U602.14, U602.3
- net at U602.11: now also U1404.3 (R3.1), U1404.4 (R4.1); no longer R630.2
- net FE_7VREF renamed FE_CTR6
- net FE_LSENS renamed FE_CTR1
- net FE_LSGND renamed FE_CTR2
- net FE_REF renamed FE_CTR3
- net FE_VOLT renamed FE_CTR0
- net M2_1 renamed FE_CTR4
- net M2_2 renamed FE_CTR5
- new net: U1403.11, U1403.14, U1403.2, U1403.7, U601.7
- new net: R1402.2, U1404.1 (R1.2), U602.14
- new net: U602.6, U602.7
- new net: R630.2, U1403.15, U1403.3
- new net: U1404.6 (R3.2), U1404.7 (R2.2)
- new net: U1404.5 (R4.2), U1404.8 (R1.2)
- new net FE_CTR7: U1403.1, U1403.16
- new net FE_CTR8: U1403.8, U1403.9
Other:
- note added: "180k/0.5%/10ppm"
- moved on the sheet: C617, C620, C624, Q601, Q602, R1401, R622, R623, R624, R625, R626, R627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

Commit message: Hardware design
Parts:
- R1401: footprint (none) -> Resistor_SMD:R_0603_1608Metric_Pad0.98x0.95mm_HandSolder
- R1411: renamed from R1402; footprint (none) -> Resistor_SMD:R_0805_2012Metric_Pad1.20x1.40mm_HandSolder
- R622: footprint Resistor_SMD:R_1206_3216Metric_Pad1.42x1.75mm_HandSolder -> Resistor_SMD:R_1206_3216Metric_Pad1.30x1.75mm_HandSolder
- R623: footprint Resistor_SMD:R_0603_1608Metric_Pad1.05x0.95mm_HandSolder -> Resistor_SMD:R_1206_3216Metric_Pad1.30x1.75mm_HandSolder
- R630: footprint Resistor_SMD:R_0603_1608Metric_Pad1.05x0.95mm_HandSolder -> Resistor_SMD:R_0603_1608Metric_Pad0.98x0.95mm_HandSolder
- renumbered C1408 to C1410, C1409 to C1411, C1410 to C1413, U1404 to U1409
