File: hardware/project/ETH1CDMM2/Power_Float.kicad_sch (KiCad schematic)
At the start: 90 parts, among them U1101 LT8330_S6, U1102 LT8330_S6, U1103 TSR1-2490, U1104 LM1117DTX-5.0/NOPB, U1105 LT3030, U1106 LM317_TO-263, U1107 LM337_TO263, U1108 TSR1-2450, U1109 LT8330_S6, U1110 LM1117DTX-3.3/NOPB, U1111 LM337_TO263

Commit message: Hardware development
Parts:
- removed C1121, C1139, C1140: 10n, Capacitor_SMD:C_0603_1608Metric_Pad1.05x0.95mm_HandSolder, symbol Device:C
- removed C1122, C1123, C1129, C1143, C1144, C1145: 4u7/50V, Capacitor_SMD:C_1206_3216Metric_Pad1.42x1.75mm_HandSolder, symbol Device:C
- removed C1124, C1125, C1128: 10u/50V, Capacitor_SMD:C_1206_3216Metric_Pad1.42x1.75mm_HandSolder, symbol Device:C
- removed C1126, C1130, C1131: 10u, Capacitor_SMD:C_0805_2012Metric_Pad1.15x1.40mm_HandSolder, symbol Device:C
- removed C1127: 4u7, Capacitor_SMD:C_0805_2012Metric_Pad1.15x1.40mm_HandSolder, symbol Device:C
- removed C1132, C1133, C1135: 1u, Capacitor_SMD:C_0603_1608Metric_Pad1.05x0.95mm_HandSolder, symbol Device:C
- removed C1134: 10u/16V, Capacitor_SMD:C_1206_3216Metric_Pad1.42x1.75mm_HandSolder, symbol Device:C
- removed C1136, C1137: 100n, Capacitor_SMD:C_0603_1608Metric_Pad1.05x0.95mm_HandSolder, symbol Device:C
- removed C1138: 1u/HC, Capacitor_SMD:C_1206_3216Metric_Pad1.42x1.75mm_HandSolder, symbol Device:C
- removed C1141: 47u/16V, Capacitor_SMD:C_1206_3216Metric_Pad1.42x1.75mm_HandSolder, symbol Device:C
- removed C1142: 4p7, Capacitor_SMD:C_0603_1608Metric_Pad1.05x0.95mm_HandSolder, symbol Device:C
- removed D1101, D1102, D1103: PMEG6010EP,115, Diode_SMD:D_SOD-128, symbol Device:D_Schottky
- removed L1102, L1103, L1105: 74489440068, ETH1CDMM2:74489440068, symbol ETH1CDMM2:74489440068
- removed L1104: TCK-141, ETH1CDMM2:TCK-141, symbol Device:L
- removed R1124: 46k4, Resistor_SMD:R_0603_1608Metric_Pad0.98x0.95mm_HandSolder, symbol Device:R
- removed R1125: 1k23, symbol Device:R
- removed R1126: 120, symbol Device:R
- removed U1101, U1102, U1109: LT8330_S6, Package_TO_SOT_SMD:TSOT-23-6_HandSoldering, symbol ETH1CDMM2:LT8330_S6
- removed U1103: TSR1-2490, ETH1CDMM2:TSR1, symbol ETH1CDMM2:TSR1-2450
- removed U1104: LM1117DTX-5.0/NOPB, Package_TO_SOT_SMD:TO-252-2, symbol ETH1CDMM2-rescue:LM1117-3.3-Regulator_Linear
- removed U1105: LT3030, Package_SO:ETSSOP-20-1EP_4.4x6.5mm_P0.65mm_EP3x4.2mm, symbol ETH1CDMM2:LT3030
- removed U1106: LM317_TO-263, Package_TO_SOT_SMD:TO-263-2, symbol Regulator_Linear:LM317_TO-263
- removed U1107, U1111: LM337_TO263, Package_TO_SOT_SMD:TO-263-2, symbol Regulator_Linear:LM337_TO263
- removed U1108: TSR1-2450, ETH1CDMM2:TSR1, symbol ETH1CDMM2:TSR1-2450
- removed U1110: LM1117DTX-3.3/NOPB, Package_TO_SOT_SMD:TO-252-2, symbol ETH1CDMM2-rescue:LM1117-3.3-Regulator_Linear
- added C212: 10u, Capacitor_SMD:C_0805_2012Metric_Pad1.15x1.40mm_HandSolder, symbol Device:C
- added C220, C221, C239, C240: 10n, Capacitor_SMD:C_0603_1608Metric_Pad1.08x0.95mm_HandSolder, symbol Device:C
- added C225, C230, C231: 10u, Capacitor_SMD:C_0805_2012Metric_Pad1.18x1.45mm_HandSolder, symbol Device:C
- added C226: 4u7, Capacitor_SMD:C_0805_2012Metric_Pad1.18x1.45mm_HandSolder, symbol Device:C
- added C232, C233: 1u, Capacitor_SMD:C_0603_1608Metric_Pad1.08x0.95mm_HandSolder, symbol Device:C
- added C236, C237: 100n, Capacitor_SMD:C_0603_1608Metric_Pad1.08x0.95mm_HandSolder, symbol Device:C
- added D1101: DFLS240, Capacitor_SMD:C_0603_1608Metric_Pad1.08x0.95mm_HandSolder, symbol Device:D
- added D1102: DFLS240, symbol Device:D
- added L1102: L, symbol Device:L
- added R205, R210: 1M, Resistor_SMD:R_0603_1608Metric_Pad0.98x0.95mm_HandSolder, symbol Device:R
- added R215: 357k, Resistor_SMD:R_0603_1608Metric_Pad0.98x0.95mm_HandSolder, symbol Device:R
- added R216: 210k, Resistor_SMD:R_0603_1608Metric_Pad0.98x0.95mm_HandSolder, symbol Device:R
- added R217, R218: 100, Resistor_SMD:R_0603_1608Metric_Pad0.98x0.95mm_HandSolder, symbol Device:R
- added R219, R220: 0R1, Resistor_SMD:R_0805_2012Metric_Pad1.15x1.40mm_HandSolder, symbol Device:R
- added U1101, U1103: ADP7182ACPZ, Package_DFN_QFN:DFN-8-1EP_3x3mm_P0.5mm_EP1.65x2.38mm_ThermalVias, symbol ETH1CDMM2:ADP7182ACPZ
- added U1102: ADP7142ARDZ, Package_SO:SOIC-8-1EP_3.9x4.9mm_P1.27mm_EP2.29x3mm, symbol Regulator_Linear:ADP7142ARDZ
- added U1104: ADP5070AREZ, Package_SO:ETSSOP-20-1EP_4.4x6.5mm_P0.65mm_EP3x4.2mm, symbol Regulator_Switching:ADP5070AREZ
- added U1105: NCV1117DT33T5G, Package_TO_SOT_SMD:TO-252-2, symbol ETH1CDMM2-rescue:LM1117-3.3-Regulator_Linear
- added U1106: NCV1117DT50RKG, Package_TO_SOT_SMD:TO-252-2, symbol ETH1CDMM2-rescue:LM1117-3.3-Regulator_Linear
- added U205: LT3030xFE#PBF, Package_SO:ETSSOP-20-1EP_4.4x6.5mm_P0.65mm_EP3x4.2mm, symbol ETH1CDMM2:LT3030
- C1101: value 10u/50V -> C; footprint Capacitor_SMD:C_1206_3216Metric_Pad1.42x1.75mm_HandSolder -> Capacitor_SMD:C_0603_1608Metric_Pad1.08x0.95mm_HandSolder
- C1102: value 10u/50V -> 1u/35V; footprint Capacitor_SMD:C_1206_3216Metric_Pad1.42x1.75mm_HandSolder -> Capacitor_SMD:C_0603_1608Metric_Pad1.08x0.95mm_HandSolder
- C1103: value 4u7/50V -> 1u/35V; footprint Capacitor_SMD:C_1206_3216Metric_Pad1.42x1.75mm_HandSolder -> Capacitor_SMD:C_0603_1608Metric_Pad1.08x0.95mm_HandSolder
- C1104: value 4u7/50V -> 10u/35V; footprint Capacitor_SMD:C_1206_3216Metric_Pad1.42x1.75mm_HandSolder -> Capacitor_SMD:C_0603_1608Metric_Pad1.08x0.95mm_HandSolder
- C1105: value 10u/50V -> 1u/35V; footprint Capacitor_SMD:C_1206_3216Metric_Pad1.42x1.75mm_HandSolder -> Capacitor_SMD:C_1206_3216Metric_Pad1.33x1.80mm_HandSolder
- C1106: value 10u/50V -> 10u/35V; footprint Capacitor_SMD:C_1206_3216Metric_Pad1.42x1.75mm_HandSolder -> Capacitor_SMD:C_1206_3216Metric_Pad1.33x1.80mm_HandSolder
- C1107: value 1u -> 1u/35V; footprint Capacitor_SMD:C_0603_1608Metric_Pad1.05x0.95mm_HandSolder -> Capacitor_SMD:C_1206_3216Metric_Pad1.33x1.80mm_HandSolder
- C1108: value 1u -> 10u/35V; footprint Capacitor_SMD:C_0603_1608Metric_Pad1.05x0.95mm_HandSolder -> Capacitor_SMD:C_1206_3216Metric_Pad1.33x1.80mm_HandSolder
- C1109: value 10u/16V -> 1u/35V; footprint Capacitor_SMD:C_1206_3216Metric_Pad1.42x1.75mm_HandSolder -> (none)
- C1110: value 1u/HC -> 1u/35V; footprint Capacitor_SMD:C_1206_3216Metric_Pad1.42x1.75mm_HandSolder -> (none)
- C1111: value 1u/HC -> 100n; footprint Capacitor_SMD:C_1206_3216Metric_Pad1.42x1.75mm_HandSolder -> Capacitor_SMD:C_0603_1608Metric_Pad1.08x0.95mm_HandSolder
- C1112: value 10u -> 47n; footprint Capacitor_SMD:C_0805_2012Metric_Pad1.15x1.40mm_HandSolder -> Capacitor_SMD:C_0603_1608Metric_Pad1.08x0.95mm_HandSolder
- C1113: value 47u/16V -> 68n; footprint Capacitor_SMD:C_1206_3216Metric_Pad1.42x1.75mm_HandSolder -> Capacitor_SMD:C_0603_1608Metric_Pad1.08x0.95mm_HandSolder
- C1114: value 4p7 -> 1u; footprint Capacitor_SMD:C_0603_1608Metric_Pad1.05x0.95mm_HandSolder -> Capacitor_SMD:C_0603_1608Metric_Pad1.08x0.95mm_HandSolder
- C1115: value 4p7 -> 100n; footprint Capacitor_SMD:C_0603_1608Metric_Pad1.05x0.95mm_HandSolder -> Capacitor_SMD:C_0603_1608Metric_Pad1.08x0.95mm_HandSolder
- C1116: value 4u7/50V -> 100n; footprint Capacitor_SMD:C_1206_3216Metric_Pad1.42x1.75mm_HandSolder -> Capacitor_SMD:C_0603_1608Metric_Pad1.08x0.95mm_HandSolder
- C1117, C1118: value 4u7/50V -> 1u; footprint Capacitor_SMD:C_1206_3216Metric_Pad1.42x1.75mm_HandSolder -> Capacitor_SMD:C_0603_1608Metric_Pad1.08x0.95mm_HandSolder
- C1119: value 4u7/50V -> 1u; footprint Capacitor_SMD:C_1206_3216Metric_Pad1.42x1.75mm_HandSolder -> (none)
- C1120: value 10n -> 1u; footprint Capacitor_SMD:C_0603_1608Metric_Pad1.05x0.95mm_HandSolder -> (none)
- L1101: value TCK-141 -> SRP7030CA-6R8M; footprint ETH1CDMM2:TCK-141 -> (none)
- R1101, R1105: value 1M -> 620k
- R1102: value 287k -> 39k
- R1103: value 1M -> 6k2
- R1104: value 287k -> 10/2W; footprint Resistor_SMD:R_0603_1608Metric_Pad0.98x0.95mm_HandSolder -> (none)
- R1106: value 1M -> 39k
- R1107: value 97k6 -> 6k2
- R1108: value 1M -> 10/2W; footprint Resistor_SMD:R_0603_1608Metric_Pad0.98x0.95mm_HandSolder -> (none)
- R1109: value 46k4 -> 10/2W; footprint Resistor_SMD:R_0603_1608Metric_Pad0.98x0.95mm_HandSolder -> (none)
- R1110: value 1M -> 12k
- R1111: value 1k6 -> 47k; footprint (none) -> Resistor_SMD:R_0603_1608Metric_Pad0.98x0.95mm_HandSolder
- R1112: value 1k6 -> 620k; footprint (none) -> Resistor_SMD:R_0603_1608Metric_Pad0.98x0.95mm_HandSolder
- R1113: value 120 -> 2M4; footprint (none) -> Resistor_SMD:R_0603_1608Metric_Pad0.98x0.95mm_HandSolder
- R1114: value 120 -> 62k; footprint (none) -> Resistor_SMD:R_0603_1608Metric_Pad0.98x0.95mm_HandSolder
- R1115: value 357k -> 39k
- R1116: value 210k -> 2M4
- R1117: value 100 -> 120k
- R1118: value 100 -> 93k
- R1119, R1120: value 0R1 -> 12k; footprint Resistor_SMD:R_0805_2012Metric_Pad1.15x1.40mm_HandSolder -> Resistor_SMD:R_0603_1608Metric_Pad0.98x0.95mm_HandSolder
- R1121: value 1M -> 3k9
- R1122: value 287k -> 3k9
- R1123: value 1M -> 1R8/2W; footprint Resistor_SMD:R_0603_1608Metric_Pad0.98x0.95mm_HandSolder -> (none)
Connections:
- net +18VF: now also C1102.1, R1101.1, U1102.1 (VOUT), U1102.2 (VOUT); no longer R1113.1
- net +1V2: now also C231.1, C233.1, C237.1, C240.1, R220.1; no longer R1120.1
- net +3.3VF: now also C1117.1, U1105.2 (VO)
- net +3.3VP: now also C230.1, C232.1, C236.1, C239.1, R219.1; no longer R1119.1
- net +5VF: now also C1118.1, C1120.1, R1121.1, R1122.1, U1105.3 (VI), U1106.2 (VO); no longer C1113.1
- net -14VF: now also C1110.2, R1112.2, U1103.1 (VOUT), U1103.2 (VOUT)
- net -18VF: now also C1105.2, R1105.2, U1101.1 (VOUT), U1101.2 (VOUT); no longer R1114.1
- net AGNDF: now also C1105.1, C1110.1, C1111.2, C1114.1, C1115.2, C1120.2, R1103.2, R1107.1, R1110.1, R1115.2, R1119.1, R1120.1, C212.2, C225.2, C226.2, C230.2, C231.2, C232.2, C233.2, C236.2, C237.2, C239.2, C240.2, L1102.2, R216.1, R217.2, R218.2, U1101.6 (GND), U1102.4 (GND), U1102.9 (GND), U1103.6 (GND), U1104.1 (PGND), U1104.15 (AGND), U1104.21 (AGND), U1104.4 (SYNC/FREQ), U1105.1 (GND), U1106.1 (GND), U205.15 (GND), U205.16 (GND), U205.21 (TP), U205.5 (GND), U205.6 (GND); no longer C1105.2, C1112.2, C1113.2, R1102.2, R1104.2, R1107.2, R1109.2, R1111.2, R1112.2, R1116.1, R1117.2, R1122.2
- net at R1101.2, R1102.1: now also U1102.3 (SENSE/ADJ)
- net THRM: now reaches C1107.1
- net THRM: now also C1109.1, R1108.2, R1109.2, U1101.4 (EN), U1101.7 (VIN), U1101.8 (VIN), U1101.9 (THRM), U1103.4 (EN), U1103.7 (VIN), U1103.8 (VIN), U1103.9 (THRM)
- net at R1104.1: now also C1104.1, R1113.1, D1101.1 (K); no longer R1103.2
- net at C1108.1: now also C1106.1, R1108.1, R1109.1, R1116.1, D1102.2 (A)
- net at C1111.1: now also U1104.14 (VREF)
- net at L1101.2: now also D1101.2 (A), U1104.2 (SW1); no longer C1106.1
- net at R1116.2: now also R1117.1, U1104.13 (FB2); no longer R1115.2
- net at R1120.2: now also C1113.1; no longer R1118.1
- net at R1110.2: now also R1111.1
- net at R1113.2: now also R1114.1, U1104.7 (FB1); no longer R1111.1
- net at R1112.1: now also R1111.2, U1103.3 (ADJ); no longer R1114.2
- net at R1123.2: now also C1115.1, C1116.1, U1104.17 (PVIN1), U1104.18 (PVINSYS), U1104.19 (PVIN2)
- net at R1121.2: now also U1104.9 (EN1); no longer R1122.1
- net +9V: now reaches R1123.1
- net +9V: now also C1119.1, C212.1, R205.1, R210.1, U1106.3 (VI), U205.11 (~{SHDN2}), U205.13 (IN), U205.14 (IN), U205.17 (IN), U205.18 (IN), U205.20 (~{SHDN1})
- removed net +24VF: C1101.1, C1102.1, C1103.1, C1104.1, C1105.1, L1101.1, R1101.1, R1103.1, R1121.1
- new net: C1113.2, U1104.12 (COMP2)
- new net: R1106.1, R1107.2
- new net: C220.1, C225.1, R215.1, R217.1, R219.2, U205.3 (OUT1), U205.4 (OUT1)
- new net: C1112.1, R1119.2
- new net: C1112.2, U1104.8 (COMP1)
- new net: C220.2, U205.2 (BYP1)
- new net: C221.1, C226.1, R218.1, R220.2, U205.10 (ADJ2), U205.7 (OUT2), U205.8 (OUT2)
- new net: R1105.1, R1106.2, U1101.3 (ADJ)
- new net: R1114.2, R1115.1
- new net: R215.2, R216.2, U205.1 (ADJ1)
- new net: R1117.2, R1118.1
- new net: C1101.1, U1102.6 (SS)
- new net: R1102.2, R1103.1
- new net: R210.2, U205.19 (PWRGD1)
- new net: D1102.1 (K), L1102.1, U1104.20 (SW2)
- new net: C1103.1, R1104.2, U1102.5 (EN), U1102.7 (VIN), U1102.8 (VIN)
- new net: R205.2, U205.12 (PWRGD2)
- new net: C221.2, U205.9 (BYP2)
- new net: R1122.2, U1104.11 (EN2)
- new net: C1114.2, U1104.16 (VREG)
- new net: L1101.1, U1104.3 (INBK)
- no-connect marks 0 -> 3

Commit message: Hardware design
Parts:
- C1108: renamed from C1119; footprint (none) -> Capacitor_SMD:C_0603_1608Metric_Pad1.08x0.95mm_HandSolder
- C1114: renamed from C1120; footprint (none) -> Capacitor_SMD:C_0603_1608Metric_Pad1.08x0.95mm_HandSolder
- C1124: renamed from C1104; footprint Capacitor_SMD:C_0603_1608Metric_Pad1.08x0.95mm_HandSolder -> Capacitor_SMD:C_1206_3216Metric_Pad1.33x1.80mm_HandSolder
- C1127: renamed from C1103; footprint Capacitor_SMD:C_0603_1608Metric_Pad1.08x0.95mm_HandSolder -> Capacitor_SMD:C_0805_2012Metric_Pad1.18x1.45mm_HandSolder
- C1128: renamed from C1107; footprint Capacitor_SMD:C_1206_3216Metric_Pad1.33x1.80mm_HandSolder -> Capacitor_SMD:C_0805_2012Metric_Pad1.18x1.45mm_HandSolder
- C1129: renamed from C1109; footprint (none) -> Capacitor_SMD:C_0805_2012Metric_Pad1.18x1.45mm_HandSolder
- C1130: renamed from C1101; value C -> 1n
- C1131: renamed from C1102; footprint Capacitor_SMD:C_0603_1608Metric_Pad1.08x0.95mm_HandSolder -> Capacitor_SMD:C_0805_2012Metric_Pad1.18x1.45mm_HandSolder
- C1132: renamed from C1105; footprint Capacitor_SMD:C_1206_3216Metric_Pad1.33x1.80mm_HandSolder -> Capacitor_SMD:C_0805_2012Metric_Pad1.18x1.45mm_HandSolder
- C1133: renamed from C1110; footprint (none) -> Capacitor_SMD:C_0805_2012Metric_Pad1.18x1.45mm_HandSolder
- C212: footprint Capacitor_SMD:C_0805_2012Metric_Pad1.15x1.40mm_HandSolder -> Capacitor_SMD:C_0805_2012Metric_Pad1.18x1.45mm_HandSolder
- D1101: renamed from D1102; footprint (none) -> ETH1CDMM2:PowerDI-123
- D1102: renamed from D1101; footprint Capacitor_SMD:C_0603_1608Metric_Pad1.08x0.95mm_HandSolder -> ETH1CDMM2:PowerDI-123
- L1101: renamed from L1102; value L -> SRP7030CA-3R3M; footprint (none) -> ETH1CDMM2:SRP7030CA
- L1102: renamed from L1101; footprint (none) -> ETH1CDMM2:SRP7030CA
- R1102: renamed from R1123; value 1R8/2W -> 1R8/.5W; footprint (none) -> Resistor_SMD:R_0805_2012Metric_Pad1.20x1.40mm_HandSolder
- R1120: renamed from R1104; value 10/2W -> 10/.5W; footprint (none) -> Resistor_SMD:R_0805_2012Metric_Pad1.20x1.40mm_HandSolder
- R1121: renamed from R1108; value 10/2W -> 10/.5W; footprint (none) -> Resistor_SMD:R_0805_2012Metric_Pad1.20x1.40mm_HandSolder
- R1122: renamed from R1109; value 10/2W -> 10/.5W; footprint (none) -> Resistor_SMD:R_0805_2012Metric_Pad1.20x1.40mm_HandSolder
- R219, R220: footprint Resistor_SMD:R_0805_2012Metric_Pad1.15x1.40mm_HandSolder -> Resistor_SMD:R_0805_2012Metric_Pad1.20x1.40mm_HandSolder
- renumbered C1118 to C1102, C1116 to C1103, C1115 to C1104, C1117 to C1105, C1112 to C1106, C1113 to C1107, C1114 to C1111, C1111 to C1117, C1106 to C1125, C1108 to C1126, R1119 to R1104, R1120 to R1105, R1121 to R1106, R1122 to R1107, R1116 to R1114, R1117 to R1115, R1118 to R1116, R1114 to R1117, R1115 to R1118, R1113 to R1119, R1101 to R1123, R1102 to R1124, R1103 to R1125, R1107 to R1126, R1106 to R1127, R1105 to R1128, R1110 to R1129, R1111 to R1130, R1112 to R1131, U1105 to U1101, U1106 to U1103, U1102 to U1105, U1101 to U1106, U1103 to U1107
Other:
- moved on the sheet: C1125, C1126, C1128, C1129, R1114, R1115, R1116
