File: hardware/project/ETH1CDMM2/Relay_Control.kicad_sch (KiCad schematic)
At the start: 5 parts, among them U603 SN74LVC1T45DBV, U604 SN74LVC1T45DBV, U605 SN74LVC1T45DBV, U606 74HCT595, U607 74HCT595

Commit message: Hardware development
Parts:
- added R301: 10k, Resistor_SMD:R_0603_1608Metric_Pad0.98x0.95mm_HandSolder, symbol Device:R
- added R302, R303, R304, R305, R306, R307, R308, R309, R310, R311, R312, R313, R314, R315, R316, R317, R318, R319: 680, Resistor_SMD:R_0603_1608Metric_Pad0.98x0.95mm_HandSolder, symbol Device:R
- added U607 (x2): 74HCT595PW, Package_SO:TSSOP-16_4.4x5mm_P0.65mm, symbol 74xx:74HCT595
- U606, U607: value 74HCT595 -> 74HCT595PW
Connections:
- net +5VF: now also U607.10 (~{SRCLR}), U607.10 (~{SRCLR}), U607.16 (VCC), U607.16 (VCC)
- net DGNDF: now also R301.2, U607.13 (~{OE}), U607.13 (~{OE}), U607.8 (GND), U607.8 (GND)
- net at U605.3 (A), U606.12 (RCLK), U607.12 (RCLK): now also R301.1, U607.12 (RCLK), U607.12 (RCLK)
- net at U607.1 (QB): now also R315.1
- net at U604.3 (A), U606.11 (SRCLK), U607.11 (SRCLK): now also U607.11 (SRCLK), U607.11 (SRCLK)
- net at U607.15 (QA): now also R314.1
- net at U607.2 (QC): now also R316.1
- net at U607.3 (QD): now also R317.1
- net at U607.4 (QE): now also R318.1
- net MS_CTR5: now reaches U607.5 (QF)
- net MS_CTR6: now reaches U607.6 (QG)
- net MS_CTR7: now reaches U607.7 (QH)
- net at U607.9 (QH'): now also U607.14 (SER)
- new net: R309.1, U607.7 (QH)
- new net: R302.1, U607.15 (QA)
- new net: R306.1, U607.4 (QE)
- new net: R319.1, U607.15 (QA)
- new net: R307.1, U607.5 (QF)
- new net: R311.1, U607.2 (QC)
- new net: R312.1, U607.3 (QD)
- new net: R310.1, U607.1 (QB)
- new net: R313.1, U607.4 (QE)
- new net: R304.1, U607.2 (QC)
- new net: R303.1, U607.1 (QB)
- new net: R305.1, U607.3 (QD)
- new net: R308.1, U607.6 (QG)
- new net: U607.14 (SER), U607.9 (QH')
- new net FE_CTR0: R302.2
- new net FE_CTR1: R303.2
- new net FE_CTR2: R304.2
- new net FE_CTR3: R305.2
- new net FE_CTR4: R306.2
- new net FE_CTR5: R307.2
- new net FE_CTR6: R308.2
- new net FE_CTR7: R309.2
- new net FE_CTR8: R319.2
- new net MS_CTR0: R314.2
- new net MS_CTR1: R315.2
- new net MS_CTR2: R316.2
- new net MS_CTR3: R317.2
- new net MS_CTR4: R318.2
- new net OHMC0: R310.2
- new net OHMC1: R311.2
- new net OHMC2: R312.2
- new net OHMC3: R313.2
- no-connect marks 1 -> 6
Other:
- moved on the sheet: U603, U604, U605, U606, U607

Commit message: Hardware design
Parts:
- renumbered R319 to R310, R310 to R311, R311 to R312, R312 to R313, R313 to R314, R314 to R315, R315 to R316, R316 to R317, R317 to R318, R318 to R319
Changed lines of the file:
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@@
         )
         (path "/be7d1fbf-8f6a-4ef0-a932-f9076baf5f6b/00000000-0000-0000-0000-0000604e8c45"
-          (reference "#PWR0312") (unit 1)
+          (reference "#PWR0313") (unit 1)
         )
       )
@@
         )
         (path "/be7d1fbf-8f6a-4ef0-a932-f9076baf5f6b/00000000-0000-0000-0000-0000604e8c45"
-          (reference "#PWR0322") (unit 1)
+          (reference "#PWR0310") (unit 1)
         )
       )
@@
         )
         (path "/be7d1fbf-8f6a-4ef0-a932-f9076baf5f6b/00000000-0000-0000-0000-0000604e8c45"
-          (reference "#PWR0314") (unit 1)
+          (reference "#PWR0319") (unit 1)
         )
       )
@@
         )
         (path "/be7d1fbf-8f6a-4ef0-a932-f9076baf5f6b/00000000-0000-0000-0000-0000604e8c45"
-          (reference "#PWR0324") (unit 1)
+          (reference "#PWR0318") (unit 1)
         )
       )
@@
         )
         (path "/be7d1fbf-8f6a-4ef0-a932-f9076baf5f6b/00000000-0000-0000-0000-0000604e8c45"
-          (reference "#PWR0320") (unit 1)
+          (reference "#PWR0323") (unit 1)
         )
       )
@@
   (symbol (lib_id "Device:R") (at 127.635 160.02 90) (unit 1)
     (in_bom yes) (on_board yes) (dnp no)
-    (property "Reference" "R319" (at 133.985 158.75 90)
+    (property "Reference" "R310" (at 133.985 158.75 90)
       (effects (font (size 1.27 1.27)))
     )
@@
       (project "ETH1CDMM2"
         (path "/be7d1fbf-8f6a-4ef0-a932-f9076baf5f6b/00000000-0000-0000-0000-0000604e8c45"
-          (reference "R319") (unit 1)
+          (reference "R310") (unit 1)
         )
       )
@@
         )
         (path "/be7d1fbf-8f6a-4ef0-a932-f9076baf5f6b/00000000-0000-0000-0000-0000604e8c45"
-          (reference "#PWR0313") (unit 1)
+          (reference "#PWR0314") (unit 1)
         )
       )
@@
         )
         (path "/be7d1fbf-8f6a-4ef0-a932-f9076baf5f6b/00000000-0000-0000-0000-0000604e8c45"
-          (reference "#PWR0317") (unit 1)
+          (reference "#PWR0322") (unit 1)
         )
       )
@@
   (symbol (lib_id "Device:R") (at 127.635 165.1 90) (unit 1)
     (in_bom yes) (on_board yes) (dnp no)
-    (property "Reference" "R311" (at 133.985 163.83 90)
+    (property "Reference" "R312" (at 133.985 163.83 90)
       (effects (font (size 1.27 1.27)))
     )
@@
       (project "ETH1CDMM2"
         (path "/be7d1fbf-8f6a-4ef0-a932-f9076baf5f6b/00000000-0000-0000-0000-0000604e8c45"
-          (reference "R311") (unit 1)
+          (reference "R312") (unit 1)
         )
       )
@@
   (symbol (lib_id "Device:R") (at 128.27 69.85 90) (unit 1)
     (in_bom yes) (on_board yes) (dnp no)
-    (property "Reference" "R314" (at 134.62 68.58 90)
+    (property "Reference" "R315" (at 134.62 68.58 90)
       (effects (font (size 1.27 1.27)))
     )
@@
       (project "ETH1CDMM2"
         (path "/be7d1fbf-8f6a-4ef0-a932-f9076baf5f6b/00000000-0000-0000-0000-0000604e8c45"
-          (reference "R314") (unit 1)
+          (reference "R315") (unit 1)
         )
       )
@@
         )
         (path "/be7d1fbf-8f6a-4ef0-a932-f9076baf5f6b/00000000-0000-0000-0000-0000604e8c45"
-          (reference "#PWR0316") (unit 1)
+          (reference "#PWR0321") (unit 1)
         )
       )
@@
         )
         (path "/be7d1fbf-8f6a-4ef0-a932-f9076baf5f6b/00000000-0000-0000-0000-0000604e8c45"
-          (reference "#PWR0315") (unit 1)
+          (reference "#PWR0320") (unit 1)
         )
       )
@@
         )
         (path "/be7d1fbf-8f6a-4ef0-a932-f9076baf5f6b/00000000-0000-0000-0000-0000604e8c45"
-          (reference "#PWR0319") (unit 1)
+          (reference "#PWR0316") (unit 1)
         )
       )
@@
         )
         (path "/be7d1fbf-8f6a-4ef0-a932-f9076baf5f6b/00000000-0000-0000-0000-0000604e8c45"
-          (reference "#PWR0318") (unit 1)
+          (reference "#PWR0315") (unit 1)
         )
       )
@@
   (symbol (lib_id "Device:R") (at 128.27 74.93 90) (unit 1)
     (in_bom yes) (on_board yes) (dnp no)
-    (property "Reference" "R316" (at 134.62 73.66 90)
+    (property "Reference" "R317" (at 134.62 73.66 90)
       (effects (font (size 1.27 1.27)))
     )
@@
       (project "ETH1CDMM2"
         (path "/be7d1fbf-8f6a-4ef0-a932-f9076baf5f6b/00000000-0000-0000-0000-0000604e8c45"
-          (reference "R316") (unit 1)
+          (reference "R317") (unit 1)
         )
       )
@@
         )
         (path "/be7d1fbf-8f6a-4ef0-a932-f9076baf5f6b/00000000-0000-0000-0000-0000604e8c45"
-          (reference "#PWR0323") (unit 1)
+          (reference "#PWR0317") (unit 1)
         )
       )
@@
   (symbol (lib_id "Device:R") (at 128.27 72.39 90) (unit 1)
     (in_bom yes) (on_board yes) (dnp no)
-    (property "Reference" "R315" (at 134.62 71.12 90)
+    (property "Reference" "R316" (at 134.62 71.12 90)
       (effects (font (size 1.27 1.27)))
     )
@@
       (project "ETH1CDMM2"
         (path "/be7d1fbf-8f6a-4ef0-a932-f9076baf5f6b/00000000-0000-0000-0000-0000604e8c45"
-          (reference "R315") (unit 1)
+          (reference "R316") (unit 1)
         )
       )
@@
   (symbol (lib_id "Device:R") (at 127.635 167.64 90) (unit 1)
     (in_bom yes) (on_board yes) (dnp no)
-    (property "Reference" "R312" (at 133.985 166.37 90)
+    (property "Reference" "R313" (at 133.985 166.37 90)
       (effects (font (size 1.27 1.27)))
     )
@@
       (project "ETH1CDMM2"
         (path "/be7d1fbf-8f6a-4ef0-a932-f9076baf5f6b/00000000-0000-0000-0000-0000604e8c45"
-          (reference "R312") (unit 1)
+          (reference "R313") (unit 1)
         )
       )
@@
   (symbol (lib_id "Device:R") (at 127.635 162.56 90) (unit 1)
     (in_bom yes) (on_board yes) (dnp no)
-    (property "Reference" "R310" (at 133.985 161.29 90)
+    (property "Reference" "R311" (at 133.985 161.29 90)
       (effects (font (size 1.27 1.27)))
     )
@@
       (project "ETH1CDMM2"
         (path "/be7d1fbf-8f6a-4ef0-a932-f9076baf5f6b/00000000-0000-0000-0000-0000604e8c45"
-          (reference "R310") (unit 1)
+          (reference "R311") (unit 1)
         )
       )
@@
   (symbol (lib_id "Device:R") (at 127.635 170.18 90) (unit 1)
     (in_bom yes) (on_board yes) (dnp no)
-    (property "Reference" "R313" (at 133.985 168.91 90)
+    (property "Reference" "R314" (at 133.985 168.91 90)
       (effects (font (size 1.27 1.27)))
     )
@@
       (project "ETH1CDMM2"
         (path "/be7d1fbf-8f6a-4ef0-a932-f9076baf5f6b/00000000-0000-0000-0000-0000604e8c45"
-          (reference "R313") (unit 1)
+          (reference "R314") (unit 1)
         )
       )
@@
   (symbol (lib_id "Device:R") (at 128.27 77.47 90) (unit 1)
     (in_bom yes) (on_board yes) (dnp no)
-    (property "Reference" "R317" (at 134.62 76.2 90)
+    (property "Reference" "R318" (at 134.62 76.2 90)
       (effects (font (size 1.27 1.27)))
     )
@@
       (project "ETH1CDMM2"
         (path "/be7d1fbf-8f6a-4ef0-a932-f9076baf5f6b/00000000-0000-0000-0000-0000604e8c45"
-          (reference "R317") (unit 1)
+          (reference "R318") (unit 1)
         )
       )
@@
         )
         (path "/be7d1fbf-8f6a-4ef0-a932-f9076baf5f6b/00000000-0000-0000-0000-0000604e8c45"
-          (reference "#PWR0311") (unit 1)
+          (reference "#PWR0312") (unit 1)
         )
       )
@@
         )
         (path "/be7d1fbf-8f6a-4ef0-a932-f9076baf5f6b/00000000-0000-0000-0000-0000604e8c45"
-          (reference "#PWR0310") (unit 1)
+          (reference "#PWR0311") (unit 1)
         )
       )
@@
         )
         (path "/be7d1fbf-8f6a-4ef0-a932-f9076baf5f6b/00000000-0000-0000-0000-0000604e8c45"
-          (reference "#PWR0321") (unit 1)
+          (reference "#PWR0324") (unit 1)
         )
       )
@@
   (symbol (lib_id "Device:R") (at 128.27 80.01 90) (unit 1)
     (in_bom yes) (on_board yes) (dnp no)
-    (property "Reference" "R318" (at 134.62 78.74 90)
+    (property "Reference" "R319" (at 134.62 78.74 90)
       (effects (font (size 1.27 1.27)))
     )
@@
       (project "ETH1CDMM2"
         (path "/be7d1fbf-8f6a-4ef0-a932-f9076baf5f6b/00000000-0000-0000-0000-0000604e8c45"
-          (reference "R318") (unit 1)
-        )
-      )
+          (reference "R319") (unit 1)
+        )
+      )
