File: hardware/project/ETH1CDMM2/ETH1CDMM2.kicad_pcb (KiCad board)
At the start: 2 copper layers, 160 x 100 mm, 431 parts, among them J1201 C64AC, J401 Conn_01x04_Male, J402 Conn_02x05, J601 Conn_02x01, J602 20021111-00010T4LF, K1201 HE3621A0510, K1202 HE3621A0510, K1203 HE3621A0510, K1204 HE3621A0510, K1205 HE3621A0510, K1206 HE3621A0510, K1502 HE3621A0510, K1503 HE3621A0510, K1504 HE3621A0510, K1505 HE3621A0510, K1506 TQ2SA-5V, Q1001 IRFR5410, Q1301 MMBFJ110, Q1303 BC857, Q1304 BC847, Q1313 MMBF4117A, Q1315 MMBF4117A, Q1401 BC847, Q1402 BC857, Q202 MMBTA55, Q203 BC847, Q401 BC857, U1001 MAX5902, U1101 ADP7182ACPZ, U1102 ADP7142ARDZ, U1103 ADP7182ACPZ, U1104 ADP5070AREZ, U1105 NCV1117DT33T5G, U1106 NCV1117DT50RKG, U1107 LT3030xFE#PBF, U1301 DG211DY+, U1302 DG211DY+, U1303 OPA2192ID, U1401 DG211DY+, U1402 DG211DY+, U1403 DG211DY+, U1404 LT5400-8, U1408 LTC1052CN8#PBF, U1409 AD711JRZ, U1410 AD711JRZ, U1411 TL431DBZ, U1412 TL431DBZ, U1501 DG211DY+, U201 DG211DY+, U202 OPA2192ID, U203 DG419DY+, U204 LT1021-7, U205 LT5400-100k-100k, U206 LM399H, U207 LT5400-5k-1k, U208 OPA177GS, U209 OPA140AID, U210 OPA177GS, U211 OPA192ID, U212 LT5400-10k-10k, U213 LM311DR, U301 SN74LVC1T45DBV, U302 SN74LVC1T45DBV, U303 SN74LVC1T45DBV, U304 74HCT595PW, U305 74HCT595PW, U306 74HCT595PW, U307 74HCT595PW, U401 SN74LVC1T45DBV, U402 SN74LVC1T45DBV, U403 ICE40HX4K-TQ144, U404 SN74LVC1T45DBV, U405 SN74LVC1T45DBV, U406 SN74LVC1T45DBV, U407 SN74LVC1T45DBV, U408 ASDMB-100.000MHZ, U409 MT25QL128ABA1ESE, U501 MT48LC16M16A2P-6A, U601 HDC1080, U602 STM32H743ZI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

Commit message: Hardware design
Parts:
- added C1101: 10u, Capacitor_SMD:C_0805_2012Metric_Pad1.18x1.45mm_HandSolder, F.Cu at (32.0, 40.8)
- added C1108: 1u, Capacitor_SMD:C_0603_1608Metric_Pad1.08x0.95mm_HandSolder, F.Cu at (31.8, 52.7)
- added C1114: 1u, Capacitor_SMD:C_0603_1608Metric_Pad1.08x0.95mm_HandSolder, F.Cu at (31.8, 55.2)
- added C1129: 1u/35V, Capacitor_SMD:C_0805_2012Metric_Pad1.18x1.45mm_HandSolder, F.Cu at (32.0, 43.8)
- added C1133: 1u/35V, Capacitor_SMD:C_0805_2012Metric_Pad1.18x1.45mm_HandSolder, F.Cu at (32.0, 46.8)
- added C703: 220p/250V, Capacitor_SMD:C_1206_3216Metric_Pad1.33x1.80mm_HandSolder, F.Cu at (44.6, 40.9)
- added C704: 220p/250V, Capacitor_SMD:C_1206_3216Metric_Pad1.33x1.80mm_HandSolder, F.Cu at (44.6, 44.3)
- added D1101: DFLS240, ETH1CDMM2:PowerDI-123, F.Cu at (32.2, 49.8)
- added D1301: BZT52B6V8-E3-18, Diode_SMD:D_SOD-123F, F.Cu at (13.8, 54.3)
- added D1302: MMSZ5229C-E3-08, Diode_SMD:D_SOD-123F, F.Cu at (13.8, 57.6)
- added D1303: BAV103, Diode_SMD:D_MiniMELF, F.Cu at (19.7, 54.3)
- added D1304: BAV103, Diode_SMD:D_MiniMELF, F.Cu at (19.7, 57.6)
- added L1001: 24S220C, ETH1CDMM2:24S220C, F.Cu at (175.3, 90.0)
- added L1101: SRP7030CA-3R3M, ETH1CDMM2:SRP7030CA, F.Cu at (112.6, 131.3)
- added L1102: SRP7030CA-6R8M, ETH1CDMM2:SRP7030CA, F.Cu at (93.2, 130.9)
- added L1501: L0805R100MPWRT, Inductor_SMD:L_0805_2012Metric_Pad1.15x1.40mm_HandSolder, F.Cu at (-0.12, 69.3)
- added L1502: L0805R100MPWRT, Inductor_SMD:L_0805_2012Metric_Pad1.15x1.40mm_HandSolder, F.Cu at (-0.12, 72.3)
- added Q1302: MMBFJ175LT1G, Package_TO_SOT_SMD:SOT-23, F.Cu at (4.70, 41.5)
- added Q1304: MMBFJ201, Package_TO_SOT_SMD:SOT-23, F.Cu at (4.70, 45.9)
- added Q1306: MMBT6520, Package_TO_SOT_SMD:SOT-23, F.Cu at (4.70, 50.4)
- added Q1307: BF823, Package_TO_SOT_SMD:SOT-23, F.Cu at (9.59, 41.5)
- added Q1308: MMBT6520, Package_TO_SOT_SMD:SOT-23, F.Cu at (-5.08, 45.0)
- added Q1309: MMBF4117, Package_TO_SOT_SMD:SOT-23, F.Cu at (9.59, 50.4)
- added Q1310: MMBT6520, Package_TO_SOT_SMD:SOT-23, F.Cu at (14.5, 41.5)
- added Q1311: MMBT6520, Package_TO_SOT_SMD:SOT-23, F.Cu at (14.5, 45.9)
- added Q1312: MMBT6520, Package_TO_SOT_SMD:SOT-23, F.Cu at (14.5, 50.4)
- added Q1313: MMBT6520, Package_TO_SOT_SMD:SOT-23, F.Cu at (19.4, 41.5)
- added Q1314: MMBT6520, Package_TO_SOT_SMD:SOT-23, F.Cu at (19.4, 45.9)
- added Q1315: MMBT6520, Package_TO_SOT_SMD:SOT-23, F.Cu at (19.4, 50.4)
- added R1001: 100k, Resistor_SMD:R_0603_1608Metric_Pad0.98x0.95mm_HandSolder, F.Cu at (31.8, 73.3)
- added R1002: 6k8/0.5W, Resistor_SMD:R_0805_2012Metric_Pad1.20x1.40mm_HandSolder, F.Cu at (27.2, 73.5)
- added R1102: 1R8/.5W, Resistor_SMD:R_0805_2012Metric_Pad1.20x1.40mm_HandSolder, F.Cu at (27.2, 40.7)
- added R1112: 0R1, Resistor_SMD:R_0805_2012Metric_Pad1.20x1.40mm_HandSolder, F.Cu at (27.2, 43.7)
- added R1113: 0R1, Resistor_SMD:R_0805_2012Metric_Pad1.20x1.40mm_HandSolder, F.Cu at (27.2, 46.6)
- added R1120: 10/.5W, Resistor_SMD:R_0805_2012Metric_Pad1.20x1.40mm_HandSolder, F.Cu at (27.2, 49.6)
- added R1121: 10/.5W, Resistor_SMD:R_0805_2012Metric_Pad1.20x1.40mm_HandSolder, F.Cu at (27.2, 52.5)
- added R1122: 10/.5W, Resistor_SMD:R_0805_2012Metric_Pad1.20x1.40mm_HandSolder, F.Cu at (27.2, 55.5)
- added R1301: 10M/.1%, Resistor_SMD:R_1206_3216Metric_Pad1.30x1.75mm_HandSolder, F.Cu at (19.5, 60.9)
- added R1302: 10M/.1%, Resistor_SMD:R_1206_3216Metric_Pad1.30x1.75mm_HandSolder, F.Cu at (19.5, 64.2)
- added R1306: 240k/.1%, Resistor_SMD:R_0603_1608Metric_Pad0.98x0.95mm_HandSolder, F.Cu at (13.2, 60.6)
- added R1307: 62k/.1%, Resistor_SMD:R_0603_1608Metric_Pad0.98x0.95mm_HandSolder, F.Cu at (13.2, 63.1)
- added R1308: 240k, Resistor_SMD:R_0805_2012Metric_Pad1.20x1.40mm_HandSolder, F.Cu at (-0.12, 40.7)
- added R1309: 196k, Resistor_SMD:R_0805_2012Metric_Pad1.20x1.40mm_HandSolder, F.Cu at (-0.12, 43.7)
- added R1310: 196k, Resistor_SMD:R_0805_2012Metric_Pad1.20x1.40mm_HandSolder, F.Cu at (-0.12, 46.6)
- added R1311: 196k, Resistor_SMD:R_0805_2012Metric_Pad1.20x1.40mm_HandSolder, F.Cu at (-0.12, 49.6)
- added R1312: 196k, Resistor_SMD:R_0805_2012Metric_Pad1.20x1.40mm_HandSolder, F.Cu at (-0.12, 52.5)
- added R1401: 100k, Resistor_SMD:R_0603_1608Metric_Pad0.98x0.95mm_HandSolder, F.Cu at (48.0, 78.2)
- added R1402: 22/.1%, Resistor_SMD:R_1206_3216Metric_Pad1.30x1.75mm_HandSolder, F.Cu at (42.9, 78.6)
- added R1403: 12k/.05%, Resistor_SMD:R_1206_3216Metric_Pad1.30x1.75mm_HandSolder, F.Cu at (42.9, 81.9)
- added R1404: 620/.05%, Resistor_SMD:R_0603_1608Metric_Pad0.98x0.95mm_HandSolder, F.Cu at (48.0, 80.8)
- added R1411: RG2012N-184-W-T1, Resistor_SMD:R_0805_2012Metric_Pad1.20x1.40mm_HandSolder, F.Cu at (42.3, 85.0)
- added R1519: 620, Resistor_SMD:R_0805_2012Metric_Pad1.20x1.40mm_HandSolder, F.Cu at (-0.12, 75.2)
- added R1521: 240k/.05%, Resistor_SMD:R_0805_2012Metric_Pad1.20x1.40mm_HandSolder, F.Cu at (-0.12, 78.2)
- added R1522: Y11215R00000B9R, Resistor_SMD:R_1206_3216Metric_Pad1.30x1.75mm_HandSolder, F.Cu at (5.23, 78.0)
- added R1523: WSR5R1000DEK, ETH1CDMM2:WSR5, F.Cu at (144.0, 64.0)
- added R1524: 240k/.05%, Resistor_SMD:R_0805_2012Metric_Pad1.20x1.40mm_HandSolder, F.Cu at (-0.12, 81.1)
- added R1525: 100k, Resistor_SMD:R_0805_2012Metric_Pad1.20x1.40mm_HandSolder, F.Cu at (-0.12, 84.1)
- added R1526: 24k, Resistor_SMD:R_0805_2012Metric_Pad1.20x1.40mm_HandSolder, F.Cu at (-0.12, 87.0)
- added R203: 4k7/.1%, Resistor_SMD:R_0603_1608Metric_Pad0.98x0.95mm_HandSolder, F.Cu at (27.1, 78.2)
- added R204: 4k7/.1%, Resistor_SMD:R_0603_1608Metric_Pad0.98x0.95mm_HandSolder, F.Cu at (27.1, 80.8)
- added R205: 0, Resistor_SMD:R_0603_1608Metric_Pad0.98x0.95mm_HandSolder, F.Cu at (27.1, 83.3)
- added R209: 62/.1%, Resistor_SMD:R_0603_1608Metric_Pad0.98x0.95mm_HandSolder, F.Cu at (27.1, 85.8)
- added R212: 6k95/.05%, Resistor_SMD:R_1206_3216Metric_Pad1.30x1.75mm_HandSolder, F.Cu at (27.9, 88.7)
- added R213: 12k/.05%, Resistor_SMD:R_0603_1608Metric_Pad0.98x0.95mm_HandSolder, F.Cu at (31.4, 78.2)
- added R214: 3k01/.1%, Resistor_SMD:R_0603_1608Metric_Pad0.98x0.95mm_HandSolder, F.Cu at (31.4, 80.8)
- added R215: 3k01/.1%, Resistor_SMD:R_0603_1608Metric_Pad0.98x0.95mm_HandSolder, F.Cu at (31.4, 83.3)
- added R220: 620/.05%, Resistor_SMD:R_0603_1608Metric_Pad0.98x0.95mm_HandSolder, F.Cu at (31.4, 85.8)
- added R221: 3k9/.05%, Resistor_SMD:R_0603_1608Metric_Pad0.98x0.95mm_HandSolder, F.Cu at (35.8, 78.2)
- added R223: 62/.1%, Resistor_SMD:R_0603_1608Metric_Pad0.98x0.95mm_HandSolder, F.Cu at (35.8, 80.8)
- added R224: 39k/.05%, Resistor_SMD:R_0603_1608Metric_Pad0.98x0.95mm_HandSolder, F.Cu at (35.8, 83.3)
- added R225: 3k9/.05%, Resistor_SMD:R_0603_1608Metric_Pad0.98x0.95mm_HandSolder, F.Cu at (35.8, 85.8)
- added R703: 1M/400V/.5W, Resistor_SMD:R_1206_3216Metric_Pad1.30x1.75mm_HandSolder, F.Cu at (44.5, 47.6)
- added R704: 1M/400V/.5W, Resistor_SMD:R_1206_3216Metric_Pad1.30x1.75mm_HandSolder, F.Cu at (44.5, 50.9)
- added R705: 24k/150V/.2W5/.1%, Resistor_SMD:R_0805_2012Metric_Pad1.20x1.40mm_HandSolder, F.Cu at (39.2, 40.7)
- added R706: 24k/150V/.2W5/.1%, Resistor_SMD:R_0805_2012Metric_Pad1.20x1.40mm_HandSolder, F.Cu at (39.2, 43.7)
- added R707: 24k/150V/.2W5/.1%, Resistor_SMD:R_0805_2012Metric_Pad1.20x1.40mm_HandSolder, F.Cu at (39.2, 46.6)
- added R710: 24k/150V/.2W5/.1%, Resistor_SMD:R_0805_2012Metric_Pad1.20x1.40mm_HandSolder, F.Cu at (39.2, 49.6)
- added R919: 1M/1kV, Resistor_SMD:R_1206_3216Metric_Pad1.30x1.75mm_HandSolder, F.Cu at (42.9, 90.2)
- added RN1301: OSOPA1002A, ETH1CDMM2:OSOP_VIS, F.Cu at (120.3, 88.6)
- added U1002: TMR6-2419WIR, ETH1CDMM2:TMR6WIR-SINGLE_TRP, F.Cu at (198.3, 133.3)
- C1003: footprint Capacitor_SMD:C_0603_1608Metric_Pad1.08x0.95mm_HandSolder -> Capacitor_SMD:C_1206_3216Metric_Pad1.33x1.80mm_HandSolder
- C1004: renamed from C1005; footprint Capacitor_SMD:C_0805_2012Metric_Pad1.18x1.45mm_HandSolder -> Capacitor_SMD:C_1812_4532Metric_Pad1.57x3.40mm_HandSolder
- C1005: renamed from C1004; footprint Capacitor_SMD:C_0805_2012Metric_Pad1.18x1.45mm_HandSolder -> Capacitor_SMD:C_1812_4532Metric_Pad1.57x3.40mm_HandSolder
- C1006: footprint Capacitor_SMD:C_0603_1608Metric_Pad1.08x0.95mm_HandSolder -> Capacitor_SMD:C_1812_4532Metric_Pad1.57x3.40mm_HandSolder
- C1124: renamed from C1104; footprint Capacitor_SMD:C_0603_1608Metric_Pad1.08x0.95mm_HandSolder -> Capacitor_SMD:C_1206_3216Metric_Pad1.33x1.80mm_HandSolder
- C1127: renamed from C1103; footprint Capacitor_SMD:C_0603_1608Metric_Pad1.08x0.95mm_HandSolder -> Capacitor_SMD:C_0805_2012Metric_Pad1.18x1.45mm_HandSolder
- C1128: renamed from C1107; footprint Capacitor_SMD:C_1206_3216Metric_Pad1.33x1.80mm_HandSolder -> Capacitor_SMD:C_0805_2012Metric_Pad1.18x1.45mm_HandSolder
- C1130: renamed from C1101; value C -> 1n
- C1131: renamed from C1102; footprint Capacitor_SMD:C_0603_1608Metric_Pad1.08x0.95mm_HandSolder -> Capacitor_SMD:C_0805_2012Metric_Pad1.18x1.45mm_HandSolder
- C1132: renamed from C1105; footprint Capacitor_SMD:C_1206_3216Metric_Pad1.33x1.80mm_HandSolder -> Capacitor_SMD:C_0805_2012Metric_Pad1.18x1.45mm_HandSolder
- D1102: renamed from D1101; footprint Capacitor_SMD:C_0603_1608Metric_Pad1.08x0.95mm_HandSolder -> ETH1CDMM2:PowerDI-123
- D201: renamed from D202; footprint Diode_SMD:D_SOD-523 -> Diode_SMD:D_SOD-123
- F1001, U501: moved to B.Cu
- Q202: value MMBTA55 -> MMBTA55-TP
- R1303, R1304: footprint Resistor_SMD:R_0603_1608Metric_Pad0.98x0.95mm_HandSolder -> Resistor_SMD:R_0805_2012Metric_Pad1.20x1.40mm_HandSolder
- R701, R702: value 24k/200V/.5W/.25% -> 24k/150V/.2W5/.1%
- moved U1101 288.3 mm to (165.1, 131.8)
- moved F1001 278.5 mm to (216.7, 135.1)
- moved U1103 272.7 mm to (149.4, 131.8)
- moved R1103 265.1 mm to (132.6, 124.8)
- moved U1102 259.6 mm to (133.7, 133.0), turned to 90 degrees
- moved R701 253.9 mm to (194.2, 73.2), turned to 180 degrees
- moved C213 246.7 mm to (112.1, 67.4), turned to 90 degrees
- moved U902 242.8 mm to (208.2, 98.9), turned to -90 degrees
- moved U903 235.2 mm to (208.2, 104.9), turned to -90 degrees
- moved U1105 231.8 mm to (93.0, 114.7)
- moved U1107 231.0 mm to (84.9, 114.8)
- moved U1106 229.9 mm to (84.9, 121.8)
- moved U1104 229.3 mm to (103.1, 131.1)
- moved U802 227.6 mm to (197.2, 87.1)
- moved J402 197.1 mm to (116.0, 102.3)
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- renumbered C1118 to C1102, C1116 to C1103, C1115 to C1104, C1117 to C1105, C1112 to C1106, C1113 to C1107, C1122 to C1109, C1123 to C1110, C1114 to C1111, C1124 to C1112, C1125 to C1113, C1126 to C1115, C1127 to C1116, C1111 to C1117, C1128 to C1118, C1129 to C1119, C1130 to C1120, C1131 to C1121, C1132 to C1122, C1133 to C1123, C1106 to C1125, C1108 to C1126, C1424 to C1408, C1417 to C1409, C1408 to C1410, C1409 to C1411, C1420 to C1412, C1410 to C1413, C1502 to C1501, C1503 to C1502, C1504 to C1503, C1501 to C1504, C202 to C201, C203 to C202, C204 to C203, C205 to C204, C206 to C205, C207 to C206, C208 to C207, C209 to C208, C210 to C209, C212 to C210, C213 to C212, C214 to C213, C215 to C214, C216 to C215, C217 to C216, C218 to C217, C219 to C218, C220 to C219, C221 to C220, C223 to C221, C224 to C223, D203 to D202, D204 to D203, D205 to D204, K1505 to K1501, K1504 to K1502, K1502 to K1504, K1506 to K1505, Q1304 to Q1305, Q203 to Q201, R1124 to R1101, R1125 to R1103, R1119 to R1104, R1120 to R1105, R1121 to R1106, R1122 to R1107, R1126 to R1108, R1127 to R1109, R1128 to R1110, R1129 to R1111, R1116 to R1114, R1117 to R1115, R1118 to R1116, R1114 to R1117, R1115 to R1118, R1113 to R1119, R1101 to R1123, R1102 to R1124, R1103 to R1125, R1107 to R1126, R1106 to R1127, R1105 to R1128, R1110 to R1129, R1111 to R1130, R1112 to R1131, R1424 to R1405, R1425 to R1406, R1426 to R1407, R1427 to R1408, R1428 to R1409, R1429 to R1410, R1515 to R1501, R1501 to R1502, R1516 to R1503, R1502 to R1504, R1517 to R1505, R1503 to R1506, R1518 to R1507, R1504 to R1508, R1519 to R1509, R1505 to R1510, R1520 to R1511, R1506 to R1512, R1521 to R1513, R1507 to R1514, R1522 to R1515, R1508 to R1516, R1509 to R1517, R1510 to R1518, R1511 to R1520, R203 to R201, R205 to R202, R207 to R206, R208 to R207, R209 to R208, R211 to R210, R212 to R211, R217 to R216, R218 to R217, R219 to R218, R220 to R219, R223 to R222, R319 to R310, R310 to R311, R311 to R312, R312 to R313, R313 to R314, R314 to R315, R315 to R316, R316 to R317, R317 to R318, R318 to R319, U1105 to U1101, U1107 to U1102, U1106 to U1103, U1102 to U1105, U1101 to U1106, U1103 to U1107, U1302 to U1301, U1301 to U1302, U1408 to U1404, U1410 to U1405, U1411 to U1406, U1412 to U1407, U1409 to U1408, U1404 to U1409, U205 to U204, U204 to U205
Connections:
- Q1305 pad 1: Net-(Q1304-B) -> Net-(Q1305-B)
- R1305 pad 2: Net-(Q1304-B) -> Net-(Q1305-B)
Other:
- outline, holes or cut-outs redrawn

Commit message: PCB design
Parts:
- added D1501: 1N4148W, Diode_SMD:D_SOD-123, B.Cu at (174.5, 67.4)
- added J101: 36107406S, ETH1CDMM2:36107406S, F.Cu at (123.1, -24.3)
- C201, C202, C203, C205, C206, C208, C209, C210, C211, C212, C215, C216, C217, C219, C220, C222, C223, C701, C702, C705, D204, R1501, R1503, R1505, R1507, R1509, R1525, R203, R210, R212, R213, R216, R218, R701, R702, R703, R704, R705, R706, R707, R708, R709, R710: moved to B.Cu
- C703, C704: footprint Capacitor_SMD:C_1206_3216Metric_Pad1.33x1.80mm_HandSolder -> Capacitor_SMD:C_0805_2012Metric_Pad1.18x1.45mm_HandSolder; moved to B.Cu
- R1522: footprint Resistor_SMD:R_1206_3216Metric_Pad1.30x1.75mm_HandSolder -> Resistor_SMD:R_2512_6332Metric_Pad1.40x3.35mm_HandSolder
- R1523: value WSR5R1000DEK -> PCS2512DR1000ET; footprint ETH1CDMM2:WSR5 -> Resistor_SMD:R_2512_6332Metric_Pad1.40x3.35mm_HandSolder
- moved U202 263.2 mm to (115.6, 68.3), turned to -90 degrees
- moved U203 257.6 mm to (109.9, 68.3), turned to 90 degrees
- moved U208 252.7 mm to (104.3, 68.3), turned to 90 degrees
- moved R702 251.8 mm to (191.8, 71.2), turned to 180 degrees
- moved C203 250.3 mm to (117.5, 68.3), turned to 90 degrees
- moved U209 250.0 mm to (99.7, 57.9), turned to 90 degrees
- moved U701 249.8 mm to (181.9, 57.7), turned to 180 degrees
- moved D204 248.5 mm to (94.9, 57.9), turned to 90 degrees
- moved D203 247.9 mm to (94.9, 57.9), turned to -90 degrees
- moved R709 247.6 mm to (191.8, 57.7), turned to 90 degrees
- moved R708 244.9 mm to (189.4, 57.7), turned to -90 degrees
- moved C202 244.6 mm to (111.8, 68.3), turned to 90 degrees
- moved C206 244.3 mm to (110.7, 60.2)
- moved U210 243.6 mm to (104.3, 77.0), turned to 90 degrees
- moved C209 242.7 mm to (109.3, 68.3), turned to -90 degrees
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