File: hardware/project/ETH1CDMM2/ETH1CDMM2.kicad_sch (KiCad schematic)
At the start: 0 parts

Commit message: Hardware development
Other:
- sheet Power float renamed Power Float
- sheet ADC ports: added none; removed FPGA_AD_RFS_OPT
- sheet Current Source ports: added OHMC[0..3]; removed none
- sheet FPGA ports: added none; removed FPGA_AD_RFS_OPT
- sheet Front End ports: added FE_CTR[0..8]; removed none
- sheet MCU ports: added SPI4_MOSI, SPI4_NSS, SPI4_SCK; removed none
- sheet Measurement Select ports: added MS_CTR[0..7]; removed none
- sheet Relay Control ports: added FE_CTR[0..8], MS_CTR[0..7], OHMC[0..3]; removed none
Changed lines of the file:
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@@
 (kicad_sch (version 20230121) (generator eeschema)
   (paper "A4")
+  (bus (pts (xy 87.63 67.31) (xy 82.55 67.31))
+    (stroke (width 0) (type default))
+  )
   (wire (pts (xy 36.83 114.3) (xy 30.48 114.3))
     (stroke (width 0) (type default))
@@
     (stroke (width 0) (type default))
   )
+  (bus (pts (xy 82.55 54.61) (xy 128.27 54.61))
+    (stroke (width 0) (type default))
+  )
   (wire (pts (xy 127 140.97) (xy 132.08 140.97))
     (stroke (width 0) (type default))
@@
     (stroke (width 0) (type default))
   )
-  (wire (pts (xy 129.54 44.45) (xy 129.54 21.59))
+  (bus (pts (xy 85.09 57.15) (xy 219.71 57.15))
+    (stroke (width 0) (type default))
+  )
+  (wire (pts (xy 124.46 44.45) (xy 124.46 21.59))
+    (stroke (width 0) (type default))
+  )
+  (bus (pts (xy 80.01 69.85) (xy 80.01 29.21))
     (stroke (width 0) (type default))
   )
@@
     (stroke (width 0) (type default))
   )
+  (bus (pts (xy 80.01 29.21) (xy 87.63 29.21))
+    (stroke (width 0) (type default))
+  )
   (wire (pts (xy 127 158.75) (xy 132.08 158.75))
     (stroke (width 0) (type default))
@@
     (stroke (width 0) (type default))
   )
+  (bus (pts (xy 73.66 72.39) (xy 87.63 72.39))
+    (stroke (width 0) (type default))
+  )
   (wire (pts (xy 215.9 91.44) (xy 219.71 91.44))
     (stroke (width 0) (type default))
@@
     (stroke (width 0) (type default))
   )
+  (bus (pts (xy 87.63 64.77) (xy 85.09 64.77))
+    (stroke (width 0) (type default))
+  )
+  (bus (pts (xy 128.27 29.21) (xy 132.08 29.21))
+    (stroke (width 0) (type default))
+  )
   (wire (pts (xy 168.91 19.05) (xy 176.53 19.05))
     (stroke (width 0) (type default))
@@
     (stroke (width 0) (type default))
   )
-  (wire (pts (xy 73.66 132.08) (xy 87.63 132.08))
+  (wire (pts (xy 127 67.31) (xy 132.08 67.31))
+    (stroke (width 0) (type default))
+  )
+  (bus (pts (xy 82.55 67.31) (xy 82.55 54.61))
     (stroke (width 0) (type default))
   )
@@
     (stroke (width 0) (type default))
   )
+  (bus (pts (xy 85.09 64.77) (xy 85.09 57.15))
+    (stroke (width 0) (type default))
+  )
   (wire (pts (xy 127 114.3) (xy 132.08 114.3))
     (stroke (width 0) (type default))
   )
+  (wire (pts (xy 127 69.85) (xy 132.08 69.85))
+    (stroke (width 0) (type default))
+  )
   (bus (pts (xy 132.08 184.15) (xy 127 184.15))
     (stroke (width 0) (type default))
@@
     (stroke (width 0) (type default))
   )
+  (bus (pts (xy 87.63 69.85) (xy 80.01 69.85))
+    (stroke (width 0) (type default))
+  )
   (wire (pts (xy 27.94 19.05) (xy 27.94 116.84))
     (stroke (width 0) (type default))
@@
     (stroke (width 0) (type default))
   )
-  (wire (pts (xy 34.29 44.45) (xy 129.54 44.45))
+  (wire (pts (xy 34.29 44.45) (xy 124.46 44.45))
+    (stroke (width 0) (type default))
+  )
+  (bus (pts (xy 128.27 54.61) (xy 128.27 29.21))
     (stroke (width 0) (type default))
   )
@@
     (stroke (width 0) (type default))
   )
-  (wire (pts (xy 129.54 21.59) (xy 132.08 21.59))
+  (wire (pts (xy 124.46 21.59) (xy 132.08 21.59))
     (stroke (width 0) (type default))
   )
@@
     (stroke (width 0) (type default))
   )
+  (wire (pts (xy 127 64.77) (xy 132.08 64.77))
+    (stroke (width 0) (type default))
+  )
   (wire (pts (xy 30.48 114.3) (xy 30.48 21.59))
     (stroke (width 0) (type default))
@@
     (stroke (width 0) (type solid))
     (fill (color 0 0 0 0.0000))
-    (property "Sheetname" "Power float" (at 176.53 136.4484 0)
+    (property "Sheetname" "Power Float" (at 176.53 136.4484 0)
       (effects (font (size 1.27 1.27)) (justify left bottom))
     )
@@
       (effects (font (size 1.27 1.27)) (justify right))
     )
-    (pin "OUT_REL[0..5]" output (at 87.63 64.77 180)
+    (pin "OUT_REL[0..5]" bidirectional (at 87.63 64.77 180)
+      (effects (font (size 1.27 1.27)) (justify left))
+    )
+    (pin "MS_CTR[0..7]" bidirectional (at 87.63 67.31 180)
+      (effects (font (size 1.27 1.27)) (justify left))
+    )
+    (pin "OHMC[0..3]" bidirectional (at 87.63 72.39 180)
+      (effects (font (size 1.27 1.27)) (justify left))
+    )
+    (pin "FE_CTR[0..8]" bidirectional (at 87.63 69.85 180)
       (effects (font (size 1.27 1.27)) (justify left))
     )
@@
       (effects (font (size 1.27 1.27)) (justify left))
     )
-    (pin "FPGA_AD_RFS_OPT" input (at 73.66 132.08 0)
-      (effects (font (size 1.27 1.27)) (justify right))
-    )
     (instances
       (project "ETH1CDMM2"
@@
       (effects (font (size 1.27 1.27)) (justify left))
     )
+    (pin "SPI4_MOSI" output (at 132.08 67.31 180)
+      (effects (font (size 1.27 1.27)) (justify left))
+    )
+    (pin "SPI4_NSS" output (at 132.08 69.85 180)
+      (effects (font (size 1.27 1.27)) (justify left))
+    )
+    (pin "SPI4_SCK" output (at 132.08 64.77 180)
+      (effects (font (size 1.27 1.27)) (justify left))
+    )
     (instances
       (project "ETH1CDMM2"
@@
       (effects (font (size 1.27 1.27)) (justify left))
     )
-    (pin "FPGA_AD_RFS_OPT" output (at 87.63 132.08 180)
-      (effects (font (size 1.27 1.27)) (justify left))
-    )
     (pin "FPGA_IO3" bidirectional (at 127 119.38 0)
       (effects (font (size 1.27 1.27)) (justify right))
@@
       (effects (font (size 1.27 1.27)) (justify left))
     )
-    (pin "OUT_REL[0..5]" input (at 219.71 35.56 180)
+    (pin "OUT_REL[0..5]" bidirectional (at 219.71 57.15 180)
       (effects (font (size 1.27 1.27)) (justify left))
     )
@@
       (effects (font (size 1.27 1.27)) (justify right))
     )
+    (pin "MS_CTR[0..7]" bidirectional (at 132.08 29.21 180)
+      (effects (font (size 1.27 1.27)) (justify left))
+    )
     (instances
       (project "ETH1CDMM2"
@@
       (effects (font (size 1.27 1.27)) (justify left))
     )
+    (pin "FE_CTR[0..8]" bidirectional (at 87.63 29.21 180)
+      (effects (font (size 1.27 1.27)) (justify left))
+    )
     (instances
       (project "ETH1CDMM2"
@@
       (effects (font (size 1.27 1.27)) (justify left))
     )
-    (instances
+    (pin "OHMC[0..3]" bidirectional (at 73.66 72.39 0)
+      (effects (font (size 1.27 1.27)) (justify right))
+    )
+    (instances

Commit message: PCB design
Parts:
- added J101: 36107406S, ETH1CDMM2:36107406S, symbol Device:RFShield_OnePiece
Connections:
- new net AGNDF: J101.1 (Shield)
Changed lines of the file:
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@@
     (stroke (width 0) (type default))
   )
+  (symbol (lib_id "ETH1CDMM2:AGNDF") (at 44.45 174.625 0) (unit 1)
+    (in_bom yes) (on_board yes) (dnp no) (fields_autoplaced)
+    (property "Reference" "#PWR0101" (at 44.45 180.975 0)
+      (effects (font (size 1.27 1.27)) hide)
+    )
+    (property "Value" "AGNDF" (at 44.45 179.07 0)
+      (effects (font (size 1.27 1.27)))
+    )
+    (property "Footprint" "" (at 44.45 174.625 0)
+      (effects (font (size 1.27 1.27)) hide)
+    )
+    (property "Datasheet" "" (at 44.45 174.625 0)
+      (effects (font (size 1.27 1.27)) hide)
+    )
+    (pin "1")
+    (instances
+      (project "ETH1CDMM2"
+        (path "/be7d1fbf-8f6a-4ef0-a932-f9076baf5f6b"
+          (reference "#PWR0101") (unit 1)
+        )
+      )
+    )
+  )
+  (symbol (lib_id "Device:RFShield_OnePiece") (at 44.45 164.465 0) (unit 1)
+    (in_bom yes) (on_board yes) (dnp no) (fields_autoplaced)
+    (property "Reference" "J101" (at 60.96 163.83 0)
+      (effects (font (size 1.27 1.27)) (justify left))
+    )
+    (property "Value" "36107406S" (at 60.96 166.37 0)
+      (effects (font (size 1.27 1.27)) (justify left))
+    )
+    (property "Footprint" "ETH1CDMM2:36107406S" (at 44.45 167.005 0)
+      (effects (font (size 1.27 1.27)) hide)
+    )
+    (property "Datasheet" "~" (at 44.45 167.005 0)
+      (effects (font (size 1.27 1.27)) hide)
+    )
+    (pin "1")
+    (instances
+      (project "ETH1CDMM2"
+        (path "/be7d1fbf-8f6a-4ef0-a932-f9076baf5f6b"
+          (reference "J101") (unit 1)
+        )
+      )
+    )
+  )
   (sheet (at 176.53 113.03) (size 39.37 17.78) (fields_autoplaced)
     (stroke (width 0) (type solid))
@@
       (effects (font (size 1.27 1.27)) (justify right))
     )
-    (pin "ADC_COMP" input (at 87.63 121.92 180)
-      (effects (font (size 1.27 1.27)) (justify left))
-    )
-    (pin "FGPA_AD_ID" output (at 87.63 114.3 180)
-      (effects (font (size 1.27 1.27)) (justify left))
-    )
-    (pin "FGPA_AD_VRH" output (at 87.63 116.84 180)
-      (effects (font (size 1.27 1.27)) (justify left))
-    )
-    (pin "FGPA_AD_IRN" output (at 87.63 119.38 180)
-      (effects (font (size 1.27 1.27)) (justify left))
-    )
-    (pin "FGPA_AD_IRP" output (at 87.63 124.46 180)
-      (effects (font (size 1.27 1.27)) (justify left))
-    )
-    (pin "FPGA_AD_IIN" output (at 87.63 127 180)
-      (effects (font (size 1.27 1.27)) (justify left))
-    )
+    (pin "ADC_COMP" input (at 87.63 127 180)
+      (effects (font (size 1.27 1.27)) (justify left))
+    )
+    (pin "FGPA_AD_ID" output (at 87.63 119.38 180)
+      (effects (font (size 1.27 1.27)) (justify left))
+    )
+    (pin "FGPA_AD_VRH" output (at 87.63 114.3 180)
+      (effects (font (size 1.27 1.27)) (justify left))
+    )
+    (pin "FGPA_AD_IRN" output (at 87.63 116.84 180)
+      (effects (font (size 1.27 1.27)) (justify left))
+    )
+    (pin "FGPA_AD_IRP" output (at 87.63 121.92 180)
+      (effects (font (size 1.27 1.27)) (justify left))
+    )
+    (pin "FPGA_AD_IIN" output (at 87.63 124.46 180)
+      (effects (font (size 1.27 1.27)) (justify left))
+    )
