File: hardware/project/ETH1CDMM2/MeasurementSelect.kicad_sch (KiCad schematic)
At the start: 35 parts, among them K1502 HE3621A0510, K1503 HE3621A0510, K1504 HE3621A0510, K1505 HE3621A0510, K1506 TQ2SA-5V, U1501 DG211

Commit message: Hardware development
Parts:
- removed L601 (x2): L0805R100MPWRT, Resistor_SMD:R_0805_2012Metric_Pad1.15x1.40mm_HandSolder, symbol ADC_Test-rescue:INDUCTOR-pspice
- added C1502, C1503, C1504: 100n, Capacitor_SMD:C_0603_1608Metric_Pad1.08x0.95mm_HandSolder, symbol Device:C
- added L1501, L1503: L0805R100MPWRT, symbol Device:L
- C610: footprint Capacitor_SMD:C_1206_3216Metric_Pad1.42x1.75mm_HandSolder -> Capacitor_SMD:C_0603_1608Metric_Pad1.08x0.95mm_HandSolder
- K1502, K1503, K1504, K1505: footprint (none) -> ETH1CDMM2:HE360_x-5050462-8
- K1506: footprint (none) -> ETH1CDMM2:SA
- R1524: value 5 -> Y11215R00000B9R
- R1525: value 0R100 -> WSR5R1000DEK
- R601, R602, R603, R604, R605, R606, R607, R608, R609, R610, R619: footprint Resistor_SMD:R_0805_2012Metric_Pad1.15x1.40mm_HandSolder -> Resistor_SMD:R_0805_2012Metric_Pad1.20x1.40mm_HandSolder
- U1501: value DG211 -> DG211DY+; footprint (none) -> Package_SO:SOIC-16_3.9x9.9mm_P1.27mm
Connections:
- net +18VF: now also C1502.1
- net +5VF: now also C1503.1
- net -18VF: now also C1504.1
- net AGNDF: now also C1502.2, C1503.2, C1504.2
- net OHM_CURR: now also L1503.2
- net at K1505.4, R619.2: now also L1503.1
- net at K1502.1, R608.1, R609.1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: now also L1501.1
- net at R619.1, R620.2: now also L1501.2
Other:
- moved on the sheet: C610, K1502A, K1502B, K1503A, K1503B, K1504A, K1504B, K1505A, K1505B, K1506, R1514, R1523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

Commit message: Hardware design
Parts:
- L1501: renamed from L1503; footprint (none) -> Inductor_SMD:L_0805_2012Metric_Pad1.15x1.40mm_HandSolder
- L1502: renamed from L1501; footprint (none) -> Inductor_SMD:L_0805_2012Metric_Pad1.15x1.40mm_HandSolder
- R1522: renamed from R1524; footprint (none) -> Resistor_SMD:R_1206_3216Metric_Pad1.30x1.75mm_HandSolder
- R1523: renamed from R1525; footprint (none) -> ETH1CDMM2:WSR5
- R1525: renamed from R1523; footprint (none) -> Resistor_SMD:R_0805_2012Metric_Pad1.20x1.40mm_HandSolder
- R1526: renamed from R1514; footprint (none) -> Resistor_SMD:R_0805_2012Metric_Pad1.20x1.40mm_HandSolder
- R619, R620, R621: footprint Resistor_SMD:R_0805_2012Metric_Pad1.15x1.40mm_HandSolder -> Resistor_SMD:R_0805_2012Metric_Pad1.20x1.40mm_HandSolder
- renumbered C1502 to C1501, C1503 to C1502, C1504 to C1503, K1505 to K1501, K1504 to K1502, K1502 to K1504, K1506 to K1505

Commit message: PCB design
Parts:
- added D1501: 1N4148W, Diode_SMD:D_SOD-123, symbol Diode:1N4148W
- R1522: footprint Resistor_SMD:R_1206_3216Metric_Pad1.30x1.75mm_HandSolder -> Resistor_SMD:R_2512_6332Metric_Pad1.40x3.35mm_HandSolder
- R1523: value WSR5R1000DEK -> PCS2512DR1000ET; footprint ETH1CDMM2:WSR5 -> Resistor_SMD:R_2512_6332Metric_Pad1.40x3.35mm_HandSolder
Connections:
- net +5VF: now also D1501.1 (K)
- net MS_CTR4: now also D1501.2 (A)
Changed lines of the file:
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@@
   (junction (at 187.96 30.48) (diameter 0) (color 0 0 0 0)
   )
+  (junction (at 177.8 124.46) (diameter 0) (color 0 0 0 0)
+  )
   (junction (at 184.15 54.61) (diameter 0) (color 0 0 0 0)
   )
@@
   )
   (junction (at 220.98 123.19) (diameter 0) (color 0 0 0 0)
+  )
+  (junction (at 195.58 124.46) (diameter 0) (color 0 0 0 0)
   )
   (junction (at 208.28 54.61) (diameter 0) (color 0 0 0 0)
@@
     (stroke (width 0) (type default))
   )
-  (wire (pts (xy 194.31 124.46) (xy 204.47 124.46))
+  (wire (pts (xy 194.31 124.46) (xy 195.58 124.46))
     (stroke (width 0) (type default))
   )
@@
     (stroke (width 0) (type default))
   )
+  (wire (pts (xy 190.5 136.525) (xy 195.58 136.525))
+    (stroke (width 0) (type default))
+  )
   (wire (pts (xy 220.98 111.76) (xy 220.98 114.3))
     (stroke (width 0) (type default))
@@
     (stroke (width 0) (type default))
   )
+  (wire (pts (xy 177.8 136.525) (xy 177.8 124.46))
+    (stroke (width 0) (type default))
+  )
   (wire (pts (xy 233.68 54.61) (xy 246.38 54.61))
     (stroke (width 0) (type default))
@@
     (stroke (width 0) (type default))
   )
+  (wire (pts (xy 195.58 124.46) (xy 204.47 124.46))
+    (stroke (width 0) (type default))
+  )
   (bus (pts (xy 29.21 26.67) (xy 29.21 24.13))
     (stroke (width 0) (type default))
@@
     (stroke (width 0) (type default))
   )
+  (wire (pts (xy 176.53 124.46) (xy 177.8 124.46))
+    (stroke (width 0) (type default))
+  )
+  (wire (pts (xy 173.99 41.91) (xy 184.15 41.91))
+    (stroke (width 0) (type default))
+  )
+  (wire (pts (xy 201.93 54.61) (xy 208.28 54.61))
+    (stroke (width 0) (type default))
+  )
+  (wire (pts (xy 16.51 36.83) (xy 26.67 36.83))
+    (stroke (width 0) (type default))
+  )
+  (wire (pts (xy 254 119.38) (xy 254 129.54))
+    (stroke (width 0) (type default))
+  )
+  (wire (pts (xy 22.86 186.69) (xy 22.86 187.96))
+    (stroke (width 0) (type default))
+  )
+  (wire (pts (xy 184.15 41.91) (xy 184.15 54.61))
+    (stroke (width 0) (type default))
+  )
+  (wire (pts (xy 261.62 54.61) (xy 269.24 54.61))
+    (stroke (width 0) (type default))
+  )
+  (wire (pts (xy 105.41 30.48) (xy 187.96 30.48))
+    (stroke (width 0) (type default))
+  )
+  (wire (pts (xy 16.51 29.21) (xy 26.67 29.21))
+    (stroke (width 0) (type default))
+  )
+  (wire (pts (xy 220.98 121.92) (xy 220.98 123.19))
+    (stroke (width 0) (type default))
+  )
+  (wire (pts (xy 208.28 21.59) (xy 201.93 21.59))
+    (stroke (width 0) (type default))
+  )
+  (wire (pts (xy 92.71 54.61) (xy 97.79 54.61))
+    (stroke (width 0) (type default))
+  )
+  (wire (pts (xy 22.86 187.96) (xy 26.67 187.96))
+    (stroke (width 0) (type default))
+  )
+  (wire (pts (xy 223.52 54.61) (xy 226.06 54.61))
+    (stroke (width 0) (type default))
+  )
+  (wire (pts (xy 20.32 161.29) (xy 20.32 160.02))
+    (stroke (width 0) (type default))
+  )
+  (wire (pts (xy 92.71 41.91) (xy 92.71 54.61))
+    (stroke (width 0) (type default))
+  )
+  (wire (pts (xy 187.96 45.72) (xy 187.96 54.61))
+    (stroke (width 0) (type default))
+  )
   (wire (pts (xy 177.8 124.46) (xy 179.07 124.46))
     (stroke (width 0) (type default))
   )
-  (wire (pts (xy 173.99 41.91) (xy 184.15 41.91))
-    (stroke (width 0) (type default))
-  )
-  (wire (pts (xy 201.93 54.61) (xy 208.28 54.61))
-    (stroke (width 0) (type default))
-  )
-  (wire (pts (xy 16.51 36.83) (xy 26.67 36.83))
-    (stroke (width 0) (type default))
-  )
-  (wire (pts (xy 254 119.38) (xy 254 129.54))
-    (stroke (width 0) (type default))
-  )
-  (wire (pts (xy 22.86 186.69) (xy 22.86 187.96))
-    (stroke (width 0) (type default))
-  )
-  (wire (pts (xy 184.15 41.91) (xy 184.15 54.61))
-    (stroke (width 0) (type default))
-  )
-  (wire (pts (xy 261.62 54.61) (xy 269.24 54.61))
-    (stroke (width 0) (type default))
-  )
-  (wire (pts (xy 105.41 30.48) (xy 187.96 30.48))
-    (stroke (width 0) (type default))
-  )
-  (wire (pts (xy 16.51 29.21) (xy 26.67 29.21))
-    (stroke (width 0) (type default))
-  )
-  (wire (pts (xy 220.98 121.92) (xy 220.98 123.19))
-    (stroke (width 0) (type default))
-  )
-  (wire (pts (xy 208.28 21.59) (xy 201.93 21.59))
-    (stroke (width 0) (type default))
-  )
-  (wire (pts (xy 92.71 54.61) (xy 97.79 54.61))
-    (stroke (width 0) (type default))
-  )
-  (wire (pts (xy 22.86 187.96) (xy 26.67 187.96))
-    (stroke (width 0) (type default))
-  )
-  (wire (pts (xy 223.52 54.61) (xy 226.06 54.61))
-    (stroke (width 0) (type default))
-  )
-  (wire (pts (xy 20.32 161.29) (xy 20.32 160.02))
-    (stroke (width 0) (type default))
-  )
-  (wire (pts (xy 92.71 41.91) (xy 92.71 54.61))
-    (stroke (width 0) (type default))
-  )
-  (wire (pts (xy 187.96 45.72) (xy 187.96 54.61))
-    (stroke (width 0) (type default))
-  )
   (bus (pts (xy 29.21 31.75) (xy 29.21 29.21))
     (stroke (width 0) (type default))
   )
+  (wire (pts (xy 195.58 136.525) (xy 195.58 124.46))
+    (stroke (width 0) (type default))
+  )
   (wire (pts (xy 194.31 111.76) (xy 220.98 111.76))
     (stroke (width 0) (type default))
@@
   )
   (wire (pts (xy 20.32 160.02) (xy 16.51 160.02))
+    (stroke (width 0) (type default))
+  )
+  (wire (pts (xy 182.88 136.525) (xy 177.8 136.525))
     (stroke (width 0) (type default))
   )
@@
       (effects (font (size 1.27 1.27)) (justify left))
     )
-    (property "Footprint" "Resistor_SMD:R_1206_3216Metric_Pad1.30x1.75mm_HandSolder" (at 219.202 118.11 90)
+    (property "Footprint" "Resistor_SMD:R_2512_6332Metric_Pad1.40x3.35mm_HandSolder" (at 219.202 118.11 90)
       (effects (font (size 1.27 1.27)) hide)
     )
@@
     )
   )
+  (symbol (lib_id "Diode:1N4148W") (at 186.69 136.525 0) (unit 1)
+    (in_bom yes) (on_board yes) (dnp no) (fields_autoplaced)
+    (property "Reference" "D1501" (at 186.69 130.81 0)
+      (effects (font (size 1.27 1.27)))
+    )
+    (property "Value" "1N4148W" (at 186.69 133.35 0)
+      (effects (font (size 1.27 1.27)))
+    )
+    (property "Footprint" "Diode_SMD:D_SOD-123" (at 186.69 140.97 0)
+      (effects (font (size 1.27 1.27)) hide)
+    )
+    (property "Datasheet" "https://www.vishay.com/docs/85748/1n4148w.pdf" (at 186.69 136.525 0)
+      (effects (font (size 1.27 1.27)) hide)
+    )
+    (property "Sim.Device" "D" (at 186.69 136.525 0)
+      (effects (font (size 1.27 1.27)) hide)
+    )
+    (property "Sim.Pins" "1=K 2=A" (at 186.69 136.525 0)
+      (effects (font (size 1.27 1.27)) hide)
+    )
+    (pin "1")
+    (pin "2")
+    (instances
+      (project "ETH1CDMM2"
+        (path "/be7d1fbf-8f6a-4ef0-a932-f9076baf5f6b/2a813b18-1d26-4bda-a5a0-c0ec48b0213c"
+          (reference "D1501") (unit 1)
+        )
+      )
+    )
+  )
   (symbol (lib_id "Device:R") (at 124.46 41.91 270) (unit 1)
     (in_bom yes) (on_board yes) (dnp no)
@@
       (effects (font (size 1.27 1.27)) (justify left))
     )
-    (property "Value" "WSR5R1000DEK" (at 223.52 130.175 0)
-      (effects (font (size 1.27 1.27)) (justify left))
-    )
-    (property "Footprint" "ETH1CDMM2:WSR5" (at 219.202 128.27 90)
+    (property "Value" "PCS2512DR1000ET" (at 223.52 130.175 0)
+      (effects (font (size 1.27 1.27)) (justify left))
+    )
+    (property "Footprint" "Resistor_SMD:R_2512_6332Metric_Pad1.40x3.35mm_HandSolder" (at 219.202 128.27 90)
       (effects (font (size 1.27 1.27)) hide)
     )
@@
     )
   )
-  (symbol (lib_id "ETH1CDMM2:+5VF") (at 177.8 124.46 90) (unit 1)
-    (in_bom yes) (on_board yes) (dnp no)
-    (property "Reference" "#PWR01512" (at 181.61 124.46 0)
-      (effects (font (size 1.27 1.27)) hide)
-    )
-    (property "Value" "+5VF" (at 173.99 124.46 90)
-      (effects (font (size 1.27 1.27)) (justify left))
-    )
-    (property "Footprint" "" (at 177.8 124.46 0)
-      (effects (font (size 1.27 1.27)) hide)
-    )
-    (property "Datasheet" "" (at 177.8 124.46 0)
-      (effects (font (size 1.27 1.27)) hide)
-    )
+  (symbol (lib_id "ETH1CDMM2:+5VF") (at 176.53 124.46 90) (unit 1)
+    (in_bom yes) (on_board yes) (dnp no)
+    (property "Reference" "#PWR01512" (at 180.34 124.46 0)
+      (effects (font (size 1.27 1.27)) hide)
+    )
+    (property "Value" "+5VF" (at 172.72 124.46 90)
+      (effects (font (size 1.27 1.27)) (justify left))
+    )
+    (property "Footprint" "" (at 176.53 124.46 0)
+      (effects (font (size 1.27 1.27)) hide)
+    )
+    (property "Datasheet" "" (at 176.53 124.46 0)
+      (effects (font (size 1.27 1.27)) hide)
+    )
